File: electronics/option_1.kicad_sch (KiCad schematic)
At the start: 0 parts

Commit message: flight back. different layout. start analog ui
Parts:
- added J17: water_sensor_conn, TerminalBlock:TerminalBlock_Xinya_XY308-2.54-6P_1x06_P2.54mm_Horizontal, symbol Connector_Generic:Conn_01x06
- added J18: Conn_01x02, Connector_Samtec_HPM_THT:Samtec_HPM-02-01-x-S_Straight_1x02_Pitch5.08mm, symbol Connector_Generic:Conn_01x02
- added J19: ~, HeavyDuty:water_sensor_rods, symbol HeavyDuty:water_sensor_rods
- added U15: ~, HeavyDuty:2_water_sensor_rods, symbol HeavyDuty:water_sesnor_binary
Connections:
- new net: J17.2 (Pin_2), J19.2 (lvl_1)
- new net: J17.3 (Pin_3), J19.3 (lvl_2)
- new net: J17.4 (Pin_4), J19.4 (lvl_3)
- new net: J17.5 (Pin_5), J19.5 (lvl_4)
- new net: J17.6 (Pin_6), J19.6 (lvl_5)
- new net: J18.2 (Pin_2), U15.2 (LVL_0)
- new net COM: J17.1 (Pin_1), J18.1 (Pin_1), J19.1 (COM), U15.1 (COM)
Other:
- note added: "round PCB shape with 6 rods in the middle"
