File: electronics/electronics.kicad_sch (KiCad schematic)
At the start: 0 parts

Commit message: from Legion
Other:
- sheet centra_control_unit renamed central_control_unit
- sheet central_control_unit ports: added +BATT, SCL, SDA, WS_COM; removed none
- sheet high_power ports: added +BATT, SCL, SDA; removed none
- sheet water_sensor ports: added COM; removed none
Changed lines of the file:
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@@
 	(generator_version "8.0")
 	(paper "A4")
+	(wire
+		(pts
+			(xy 88.9 54.61) (xy 101.6 54.61)
+		)
+		(stroke
+			(width 0)
+			(type default)
+		)
+	)
+	(wire
+		(pts
+			(xy 88.9 63.5) (xy 101.6 63.5)
+		)
+		(stroke
+			(width 0)
+			(type default)
+		)
+	)
+	(wire
+		(pts
+			(xy 88.9 67.31) (xy 101.6 67.31)
+		)
+		(stroke
+			(width 0)
+			(type default)
+		)
+	)
 	(rectangle
 		(start 191.516 78.74)
@@
 	)
 	(sheet
-		(at 63.5 39.37)
-		(size 66.04 35.56)
+		(at 101.6 50.8)
+		(size 25.4 25.4)
 		(fields_autoplaced yes)
 		(stroke
@@
 			(color 255 231 58 1.0000)
 		)
-		(property "Sheetname" "centra_control_unit"
-			(at 63.5 38.6584 0)
+		(property "Sheetname" "central_control_unit"
+			(at 101.6 50.0884 0)
 			(effects
 				(font
@@
 		)
 		(property "Sheetfile" "centra_control_unit.kicad_sch"
-			(at 63.5 75.5146 0)
+			(at 101.6 76.7846 0)
 			(effects
 				(font
@@
 				)
 				(justify left top)
+			)
+		)
+		(pin "+BATT" input
+			(at 101.6 54.61 180)
+			(effects
+				(font
+					(size 1.27 1.27)
+				)
+				(justify left)
+			)
+		)
+		(pin "SCL" passive
+			(at 101.6 67.31 180)
+			(effects
+				(font
+					(size 1.27 1.27)
+				)
+				(justify left)
+			)
+		)
+		(pin "SDA" passive
+			(at 101.6 63.5 180)
+			(effects
+				(font
+					(size 1.27 1.27)
+				)
+				(justify left)
+			)
+		)
+		(pin "WS_COM" passive
+			(at 127 68.58 0)
+			(effects
+				(font
+					(size 1.27 1.27)
+				)
+				(justify right)
 			)
 		)
@@
 			)
 		)
+		(pin "COM" passive
+			(at 107.95 167.64 0)
+			(effects
+				(font
+					(size 1.27 1.27)
+				)
+				(justify right)
+			)
+		)
 		(instances
 			(project "electronics"
@@
 	)
 	(sheet
-		(at 203.2 128.27)
-		(size 12.7 12.7)
+		(at 63.5 50.8)
+		(size 25.4 25.4)
 		(fields_autoplaced yes)
 		(stroke
@@
 		)
 		(property "Sheetname" "high_power"
-			(at 203.2 127.5584 0)
+			(at 63.5 50.0884 0)
 			(effects
 				(font
@@
 		)
 		(property "Sheetfile" "high_power.kicad_sch"
-			(at 203.2 141.5546 0)
+			(at 63.5 76.7846 0)
 			(effects
 				(font
@@
 		)
 		(property "exclude" ""
-			(at 203.2 128.27 0)
+			(at 63.5 50.8 0)
 			(effects
 				(font
@@
 			)
 		)
+		(pin "SDA" bidirectional
+			(at 88.9 63.5 0)
+			(effects
+				(font
+					(size 1.27 1.27)
+				)
+				(justify right)
+			)
+		)
+		(pin "SCL" bidirectional
+			(at 88.9 67.31 0)
+			(effects
+				(font
+					(size 1.27 1.27)
+				)
+				(justify right)
+			)
+		)
+		(pin "+BATT" output
+			(at 88.9 54.61 0)
+			(effects
+				(font
+					(size 1.27 1.27)
+				)
+				(justify right)
+			)
+		)

Commit message: hss GPIO implemented, compiling fine
Other:
- company: (none) -> MK Electronics
- title: (none) -> camper_controller
Changed lines of the file:
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@@
 	(generator_version "8.0")
 	(paper "A4")
+	(title_block
+		(title "camper_controller")
+		(date "2024-12-30")
+		(rev "0")
+		(company "MK Electronics")
+	)
 	(wire
 		(pts

Commit message: flight back. different layout. start analog ui
Other:
- added sheet analog_ui (analog_ui.kicad_sch)
Changed lines of the file:
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@@
 	(rectangle
 		(start 191.516 78.74)
-		(end 227.076 100.33)
+		(end 250.19 115.57)
 		(stroke
 			(width 0)
@@
 				)
 			)
+		)
+	)
+	(sheet
+		(at 200.66 90.17)
+		(size 29.21 19.05)
+		(fields_autoplaced yes)
+		(stroke
+			(width 0.1524)
+			(type solid)
+		)
+		(fill
+			(color 0 0 0 0.0000)
+		)
+		(property "Sheetname" "analog_ui"
+			(at 200.66 89.4584 0)
+			(effects
+				(font
+					(size 1.27 1.27)
+				)
+				(justify left bottom)
+			)
+		)
+		(property "Sheetfile" "analog_ui.kicad_sch"
+			(at 200.66 109.8046 0)
+			(effects
+				(font
+					(size 1.27 1.27)
+				)
+				(justify left top)
+			)
+		)
+		(instances
+			(project "electronics"
+				(path "/eeb1234c-eae0-4ac6-a30d-2a978d66d889"
+					(page "14")
+				)
+			)

Commit message: no tracks, but placement looks good
Other:
- sheet central_control_unit ports: added none; removed +BATT, WS_COM
- sheet high_power ports: added none; removed +BATT
- sheet water_sensor ports: added none; removed COM
Changed lines of the file:
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@@
-	(wire
-		(pts
-			(xy 88.9 54.61) (xy 101.6 54.61)
-		)
-		(stroke
-			(width 0)
-			(type default)
-		)
-	)
 	(wire
 		(pts
@@
 			)
 		)
-		(pin "+BATT" input
-			(at 101.6 54.61 180)
-			(effects
-				(font
-					(size 1.27 1.27)
-				)
-				(justify left)
-			)
-		)
 		(pin "SCL" passive
 			(at 101.6 67.31 180)
@@
 				)
 				(justify left)
-			)
-		)
-		(pin "WS_COM" passive
-			(at 127 68.58 0)
-			(effects
-				(font
-					(size 1.27 1.27)
-				)
-				(justify right)
 			)
 		)
@@
 			)
 		)
-		(pin "COM" passive
-			(at 107.95 167.64 0)
-			(effects
-				(font
-					(size 1.27 1.27)
-				)
-				(justify right)
-			)
-		)
 		(instances
 			(project "electronics"
@@
 			(effects
 				(font
-					(size 1.27 1.27)
-				)
-				(justify right)
-			)
-		)
-		(pin "+BATT" output
-			(at 88.9 54.61 0)
-			(effects
-				(font
