File: electronics/centra_control_unit.kicad_sch (KiCad schematic)
At the start: 12 parts, among them U14 CD74HC4067SM, U15 TCA9555PWR, U18 SN74LV4051A, U19 ESP32-C6-MINI-1/U

Commit message: from dell
Parts:
- removed U19: ESP32-C6-MINI-1/U, PCM_Espressif:ESP32-C6-MINI-1, symbol Espressif:ESP32-C6-MINI-1/U
- added U16: MAX485E, symbol Interface_UART:MAX485E
- added U5: ESP32-S3-MINI-1, RF_Module:ESP32-S2-MINI-1U, symbol Espressif:ESP32-S3-MINI-1
- D1, D13, D14: footprint (none) -> LED_SMD:LED_1812_4532Metric_Pad1.30x3.40mm_HandSolder
Connections:
- net water_sensors_logic/WS_ENABLE is gone; now on net water_sensors_logic/WS_LVL_25%: U15.4 (P00)
- net +3.3V: now also U5.3 (3V3); no longer U15.24 (VCC)
- net GND_LP: now also U5.1 (GND), U5.2 (GND), U5.42 (GND), U5.43 (GND), U5.46 (GND), U5.47 (GND), U5.48 (GND), U5.49 (GND), U5.50 (GND), U5.51 (GND), U5.52 (GND), U5.53 (GND), U5.54 (GND), U5.55 (GND), U5.56 (GND), U5.57 (GND), U5.58 (GND), U5.59 (GND), U5.60 (GND), U5.61 (GND), U5.62 (GND), U5.63 (GND), U5.64 (GND), U5.65 (GND); no longer U15.12 (GND), U15.2 (A1), U15.21 (A0), U15.3 (A2)
- net SCL: no longer U15.22 (SCL)
- net SDA: no longer U15.23 (SDA)
- net digital_switching/CH1_DEN: no longer U15.11 (P07)
- net digital_switching/CH1_IN: no longer U15.10 (P06)
- net digital_switching/CH2_DEN: no longer U15.14 (P11)
- net digital_switching/CH2_IN: no longer U15.13 (P10)
- net digital_switching/CH3_DEN: no longer U15.16 (P13)
- net digital_switching/CH3_IN: no longer U15.15 (P12)
- net digital_switching/CH4_DEN: no longer U15.18 (P15)
- net digital_switching/CH4_IN: no longer U15.17 (P14)
- net digital_switching/CH5_DEN: no longer U15.20 (P17)
- net digital_switching/CH5_IN: no longer U15.19 (P16)
- net water_sensors_logic/GREY_WATER_FULL: now also U15.8 (P04); no longer U15.9 (P05)
- net water_sensors_logic/WS_LVL_100%: now also U15.7 (P03); no longer U15.8 (P04)
- net water_sensors_logic/WS_LVL_25%: no longer U15.5 (P01)
- net water_sensors_logic/WS_LVL_50%: now also U15.5 (P01); no longer U15.6 (P02)
- net water_sensors_logic/WS_LVL_75%: now also U15.6 (P02); no longer U15.7 (P03)
- new net ac_detect: U15.9 (P05)
- new net relay_out: U15.10 (P06)
Other:
- added sheet analog_ui_control (analog_ui_control.kicad_sch)
- sheet water_sensors_logic ports: added none; removed WS_ENABLE
- moved on the sheet: C10, D1, D13, D14, R27, R33, R34
