File: electronics/high_power.kicad_sch (KiCad schematic)
At the start: 12 parts, among them J5 Conn_01x02, J6 Conn_01x02, J7 Conn_01x02, J8 Conn_01x02

Commit message: from Legion
Parts:
- removed BT1: Battery, symbol Device:Battery
- removed BusBar1: ~, HeavyDuty:busbar-20mm, symbol HeavyDuty:BusBarConn
- removed BusBar2, BusBar3, BusBar4: ~, HeavyDuty:busbar-15mm, symbol HeavyDuty:BusBarConn
- removed J5, J6, J7, J8: Conn_01x02, symbol Connector_Generic:Conn_01x02
- added Battery1, Inverter1: ~, HeavyDuty:high_current_pad, symbol HeavyDuty:BusBarConn
- added C5, C6, C7, C8: 1uF, Capacitor_SMD:C_0805_2012Metric_Pad1.18x1.45mm_HandSolder, symbol Device:C_Small
- added F1, F2, F4: 20A, HeavyDuty:ATO_fuse_holder, symbol Device:Fuse
- added J4: Chargers_Conn, HeavyDuty:3p_terminal, symbol Connector_Generic:Conn_01x03
- added J5: 12V_BusBar, HeavyDuty:half_busbar-15mm, symbol HeavyDuty:BusBarConn
- added J6: GND_Busbar, HeavyDuty:half_busbar-15mm, symbol HeavyDuty:BusBarConn
- added MH1, MH2, MH3, MH4: MH, MountingHole:MountingHole_3.2mm_M3_ISO7380_Pad_TopBottom, symbol Mechanical:MountingHole_Pad
- added Q1: Q_PMOS_GDS, Package_TO_SOT_SMD:TO-252-3_TabPin2, symbol Device:Q_PMOS_GDS
- added R10, R11, R12, R13, R7, R9: 10 ohm, Resistor_SMD:R_0805_2012Metric_Pad1.20x1.40mm_HandSolder, symbol Device:R_Small
- added R14, R15: 4.7k, Resistor_SMD:R_1206_3216Metric_Pad1.30x1.75mm_HandSolder, symbol Device:R
- added R16: 5k, Resistor_SMD:R_0805_2012Metric_Pad1.20x1.40mm_HandSolder, symbol Device:R
- added U11: INA3221, Package_DFN_QFN:Texas_RGV0016A_VQFN-16-1EP_4x4mm_P0.65mm_EP2.1x2.1mm, symbol Power_Management:INA3221
Connections:
- net +BATT: now also R5.4, R6.4, R8.4, J5.1
- net at R6.1: now also F1.1, F2.1, F4.1
- net RSH6_HI: now reaches R6.2
- net RSH6_HI: now also R7.1
- net RSH6_LO: now reaches R6.3
- net RSH6_LO: now also R9.1
- net at R8.1: now also Inverter1.1
- net at R5.1: now also Battery1.1
- net RSH5_HI: now reaches R5.2
- net RSH5_HI: now also R12.1
- net RSH5_LO: now reaches R5.3
- net RSH5_LO: now also R13.1
- net RSH8_HI: now reaches R8.2
- net RSH8_HI: now also R10.1
- net RSH8_LO: now reaches R8.3
- net RSH8_LO: now also R11.1
- new net: C5.1, R12.2, U11.2 (IN+3)
- new net: Q1.1 (G), R16.2
- new net: C5.2, R13.2, U11.1 (IN-3)
- new net: C7.2, R9.2, U11.11 (IN-1)
- new net: C7.1, R7.2, U11.12 (IN+1)
- new net: C6.2, R11.2, U11.14 (IN-2)
- new net: C6.1, R10.2, U11.15 (IN+2)
- new net: F1.2, J4.2 (Pin_2)
- new net: F2.2, J4.3 (Pin_3)
- new net: F4.2, J4.1 (Pin_1), Q1.2 (D)
- new net +3.3V: C8.2, R14.2, R15.2, U11.4 (VS)
- new net GND: C8.1, J6.1, MH1.1, MH2.1, MH3.1, MH4.1, R16.1, U11.3 (GND), U11.5 (A0)
- new net SCL: R15.1, U11.6 (SCL)
- new net SDA: R14.1, U11.7 (SDA)
- no-connect marks 0 -> 6
Other:
- note added: "12V Power Monitoring"
- note added: "Grid charger"
- note removed: "DC Distribution Box"
- note removed: "Shunt Resistor"
- moved on the sheet: R6, R8

Commit message: hss GPIO implemented, compiling fine
Parts:
- R14: value 4.7k -> 4.7k
Changed lines of the file:
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@@
 			)
 		)
-		(property "Value" "4.7k	"
+		(property "Value" "4.7k"
 			(at 260.35 122.174 90)
 			(effects

Commit message: porady od MichalaG
Changed lines of the file:
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@@
 		)
 	)
-	(text_box "For bolts use Bellaville washers or similar\n\nhttps://electronics.stackexchange.com/questions/649672/aluminum-bus-bars-connection-to-pcb\n\nbusbar fixing to PCB: https://www.mouser.pl/ProductDetail/PEM/KF2-M5-ET?qs=l4Gc20tDgJJBILUPfp%252BXpw%3D%3D\nscrew-like stud: PEM HFHB-M5-15X\n"
+	(text_box "For bolts use Bellaville washers or similar\n\nhttps://electronics.stackexchange.com/questions/649672/aluminum-bus-bars-connection-to-pcb\n\nbusbar fixing to PCB: https://www.mouser.pl/ProductDetail/PEM/KF2-M5-ET?qs=l4Gc20tDgJJBILUPfp%252BXpw%3D%3D\nscrew-like stud: PEM HFHB-M5-15X\n\nconnector options: https://www.lcsc.com/datasheet/lcsc_datasheet_2303311800_Cixi-Kefa-Elec-KF78CM-13-0-6P_C964690.pdf\nhttps://www.lcsc.com/product-detail/PCB-Welding-Terminal_SAMZO-91186400M5_C32710810.html\n"
 		(exclude_from_sim no)
 		(at 203.2 25.4 0)
@@
 		)
 		(instances
-			(project ""
+			(project "electronics"
 				(path "/eeb1234c-eae0-4ac6-a30d-2a978d66d889/da888cb1-ed89-4b09-bf89-340f462f0940"
 					(reference "R16")
@@
 		)
 		(instances
-			(project ""
+			(project "electronics"
 				(path "/eeb1234c-eae0-4ac6-a30d-2a978d66d889/da888cb1-ed89-4b09-bf89-340f462f0940"
 					(reference "MH1")
@@
 		)
 		(instances
-			(project ""
+			(project "electronics"
 				(path "/eeb1234c-eae0-4ac6-a30d-2a978d66d889/da888cb1-ed89-4b09-bf89-340f462f0940"
 					(reference "R5")
@@
 		)
 		(instances
-			(project ""
+			(project "electronics"
 				(path "/eeb1234c-eae0-4ac6-a30d-2a978d66d889/da888cb1-ed89-4b09-bf89-340f462f0940"
 					(reference "Q1")
@@
 		)
 		(instances
-			(project ""
+			(project "electronics"
 				(path "/eeb1234c-eae0-4ac6-a30d-2a978d66d889/da888cb1-ed89-4b09-bf89-340f462f0940"
 					(reference "J4")

Commit message: lisbon flight changes
Parts:
- removed J4: Chargers_Conn, HeavyDuty:3p_terminal, symbol Connector_Generic:Conn_01x03
- removed Q1: Q_PMOS_GDS, Package_TO_SOT_SMD:TO-252-3_TabPin2, symbol Device:Q_PMOS_GDS
- removed R16: 5k, Resistor_SMD:R_0805_2012Metric_Pad1.20x1.40mm_HandSolder, symbol Device:R
- added FB1: FerriteBead 47Ohm, symbol Device:FerriteBead
- added J12, J4, J8: Conn_01x01, symbol Connector_Generic:Conn_01x01
Connections:
- net GND: no longer J6.1, U11.3 (GND), U11.5 (A0)
- net at F1.2: now also J8.1 (Pin_1)
- net at F2.2: now also J12.1 (Pin_1)
- net at F4.2: now also J4.1 (Pin_1)
- new net GND_HP: FB1.1, J6.1
- new net GND_LP: FB1.2, U11.3 (GND), U11.5 (A0)
Other:
- moved on the sheet: F1, F2, F4, J6

Commit message: flight back. different layout. start analog ui
Parts:
- removed FB1: FerriteBead 47Ohm, symbol Device:FerriteBead
- removed J5: 12V_BusBar, HeavyDuty:half_busbar-15mm, symbol HeavyDuty:BusBarConn
- added F3, F5: 20A, HeavyDuty:ATO_fuse_holder, symbol Device:Fuse
- added J23, J24: Conn_01x01, HeavyDuty:keystone_m3_screw_terminal_vertical, symbol Connector_Generic:Conn_01x01
- added Q2: AON6407-HXZ, Package_TO_SOT_SMD:SOT-23, symbol Transistor_FET:BSS83P
- Battery1: footprint HeavyDuty:high_current_pad -> HeavyDuty:small_busbar-15mm
- J12, J4, J8: footprint (none) -> HeavyDuty:keystone_m3_screw_terminal_vertical
- J6: footprint HeavyDuty:half_busbar-15mm -> HeavyDuty:small_busbar-15mm
Connections:
- net +BATT: now also F3.1, F5.1
- net GND: no longer C8.1
- net GND_LP: now also C8.1
- new net: F5.2, J24.1 (Pin_1)
- new net: F3.2, J23.1 (Pin_1)
Other:
- moved on the sheet: F1, F2, F4

Commit message: no tracks, but placement looks good
Connections:
- net GND is gone; now on net GND_HP: MH1.1, MH2.1, MH3.1, MH4.1
- net +BATT renamed V_Bat
Changed lines of the file:
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@@
+	(wire
+		(pts
+			(xy 116.84 63.5) (xy 147.32 63.5)
+		)
+		(stroke
+			(width 0)
+			(type default)
+		)
+	)
 	(wire
 		(pts
@@
 		(pts
 			(xy 71.12 140.97) (xy 106.68 140.97)
-		)
-		(stroke
-			(width 0)
-			(type default)
-		)
-	)
-	(wire
-		(pts
-			(xy 144.78 63.5) (xy 116.84 63.5)
 		)
 		(stroke
@@
 	)
 	(label "V_Bat"
-		(at 142.24 63.5 180)
+		(at 144.78 63.5 180)
 		(fields_autoplaced yes)
 		(effects
@@
 		)
 	)
+	(label "HP_Bus"
+		(at 114.3 96.52 0)
+		(fields_autoplaced yes)
+		(effects
+			(font
+				(size 1.27 1.27)
+				(color 255 52 64 1)
+			)
+			(justify left bottom)
+		)
+	)
 	(label "RSH5_LO"
 		(at 176.53 138.43 0)
@@
 			)
 			(justify left bottom)
+		)
+	)
+	(global_label "V_Bat"
+		(shape passive)
+		(at 147.32 63.5 0)
+		(fields_autoplaced yes)
+		(effects
+			(font
+				(size 1.27 1.27)
+			)
+			(justify left)
+		)
+		(property "Intersheetrefs" "${INTERSHEET_REFS}"
+			(at 154.3948 63.5 0)
+			(effects
+				(font
+					(size 1.27 1.27)
+				)
+				(justify left)
+				(hide yes)
+			)
 		)
 	)
@@
 		(shape bidirectional)
 		(at 273.05 128.27 0)
-		(fields_autoplaced yes)
-		(effects
-			(font
-				(size 1.27 1.27)
-			)
-			(justify left)
-		)
-	)
-	(hierarchical_label "+BATT"
-		(shape output)
-		(at 144.78 63.5 0)
 		(fields_autoplaced yes)
 		(effects
@@
 	)
 	(symbol
-		(lib_name "GND_1")
-		(lib_id "power:GND")
-		(at 130.81 180.34 0)
-		(unit 1)
-		(exclude_from_sim no)
-		(in_bom yes)
-		(on_board yes)
-		(dnp no)
-		(fields_autoplaced yes)
-		(property "Reference" "#PWR08"
-			(at 130.81 186.69 0)
-			(effects
-				(font
-					(size 1.27 1.27)
-				)
-				(hide yes)
-			)
-		)
-		(property "Value" "GND"
-			(at 130.81 185.42 0)
-			(effects
-				(font
-					(size 1.27 1.27)
-				)
-			)
-		)
-		(property "Footprint" ""
-			(at 130.81 180.34 0)
-			(effects
-				(font
-					(size 1.27 1.27)
-				)
-				(hide yes)
-			)
-		)
-		(property "Datasheet" ""
-			(at 130.81 180.34 0)
-			(effects
-				(font
-					(size 1.27 1.27)
-				)
-				(hide yes)
-			)
-		)
-		(property "Description" "Power symbol creates a global label with name \"GND\" , ground"
-			(at 130.81 180.34 0)
-			(effects
-				(font
-					(size 1.27 1.27)
-				)
-				(hide yes)
-			)
-		)
-		(pin "1"
-		)
-		(instances
-			(project "electronics"
-				(path "/eeb1234c-eae0-4ac6-a30d-2a978d66d889/da888cb1-ed89-4b09-bf89-340f462f0940"
-					(reference "#PWR08")
-					(unit 1)
-				)
-			)
-		)
-	)
-	(symbol
 		(lib_id "Connector_Generic:Conn_01x01")
 		(at 66.04 140.97 180)
@@
 					(unit 1)
 				)
+			)
+		)
+	)
+	(symbol
+		(lib_id "power:GND1")
+		(at 130.81 180.34 0)
+		(unit 1)
+		(exclude_from_sim no)
+		(in_bom yes)
+		(on_board yes)
+		(dnp no)
+		(fields_autoplaced yes)
+		(property "Reference" "#PWR07"
+			(at 130.81 186.69 0)
+			(effects
+				(font
+					(size 1.27 1.27)
+				)
+				(hide yes)
+			)
+		)
+		(property "Value" "GND_HP"
+			(at 130.81 185.42 0)
+			(effects
+				(font
+					(size 1.27 1.27)
+				)
+			)
+		)
+		(property "Footprint" ""
+			(at 130.81 180.34 0)
+			(effects
+				(font
+					(size 1.27 1.27)
+				)
+				(hide yes)
+			)
+		)
+		(property "Datasheet" ""
+			(at 130.81 180.34 0)
+			(effects
+				(font
+					(size 1.27 1.27)
+				)
+				(hide yes)
+			)
+		)
+		(property "Description" "Power symbol creates a global label with name \"GND1\" , ground"
+			(at 130.81 180.34 0)
+			(effects
+				(font
+					(size 1.27 1.27)
+				)
+				(hide yes)
+			)
+		)
+		(pin "1"
+		)
+		(instances
+			(project "electronics"
+				(path "/eeb1234c-eae0-4ac6-a30d-2a978d66d889/da888cb1-ed89-4b09-bf89-340f462f0940"
+					(reference "#PWR07")
+					(unit 1)
+				)

Commit message: add some lcsc and TME part numbers
Connections:
- net V_Bat renamed +12V
Changed lines of the file:
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@@
 	(wire
 		(pts
-			(xy 116.84 63.5) (xy 147.32 63.5)
+			(xy 116.84 63.5) (xy 153.67 63.5)
 		)
 		(stroke
@@
 		)
 	)
-	(global_label "V_Bat"
-		(shape passive)
-		(at 147.32 63.5 0)
-		(fields_autoplaced yes)
-		(effects
-			(font
-				(size 1.27 1.27)
-			)
-			(justify left)
-		)
-		(property "Intersheetrefs" "${INTERSHEET_REFS}"
-			(at 154.3948 63.5 0)
-			(effects
-				(font
-					(size 1.27 1.27)
-				)
-				(justify left)
-				(hide yes)
-			)
-		)
-	)
 	(hierarchical_label "SDA"
 		(shape bidirectional)
@@
 					(unit 1)
 				)
+			)
+		)
+	)
+	(symbol
+		(lib_id "power:+12V")
+		(at 153.67 63.5 0)
+		(unit 1)
+		(exclude_from_sim no)
+		(in_bom yes)
+		(on_board yes)
+		(dnp no)
+		(fields_autoplaced yes)
+		(property "Reference" "#PWR054"
+			(at 153.67 67.31 0)
+			(effects
+				(font
+					(size 1.27 1.27)
+				)
+				(hide yes)
+			)
+		)
+		(property "Value" "+12V"
+			(at 153.67 58.42 0)
+			(effects
+				(font
+					(size 1.27 1.27)
+				)
+			)
+		)
+		(property "Footprint" ""
+			(at 153.67 63.5 0)
+			(effects
+				(font
+					(size 1.27 1.27)
+				)
+				(hide yes)
+			)
+		)
+		(property "Datasheet" ""
+			(at 153.67 63.5 0)
+			(effects
+				(font
+					(size 1.27 1.27)
+				)
+				(hide yes)
+			)
+		)
+		(property "Description" "Power symbol creates a global label with name \"+12V\""
+			(at 153.67 63.5 0)
+			(effects
+				(font
+					(size 1.27 1.27)
+				)
+				(hide yes)
+			)
+		)
+		(pin "1"
+		)
+		(instances
+			(project "electronics"
+				(path "/eeb1234c-eae0-4ac6-a30d-2a978d66d889/da888cb1-ed89-4b09-bf89-340f462f0940"
+					(reference "#PWR054")
+					(unit 1)
+				)

Commit message: from dell
Parts:
- removed Battery1: ~, HeavyDuty:small_busbar-15mm, symbol HeavyDuty:BusBarConn
- removed Inverter1: ~, HeavyDuty:high_current_pad, symbol HeavyDuty:BusBarConn
- removed J6: GND_Busbar, HeavyDuty:small_busbar-15mm, symbol HeavyDuty:BusBarConn
- removed Q2: AON6407-HXZ, Package_TO_SOT_SMD:SOT-23, symbol Transistor_FET:BSS83P
- added GND_Conn1: ~, HeavyDuty:small_busbar-15mm, symbol HeavyDuty:BusBarConn
- added J14: Conn_GND, HeavyDuty:keystone_m3_screw_terminal_vertical, symbol Connector_Generic:Conn_01x01
- added J15: Battery_Conn, HeavyDuty:keystone_m3_screw_terminal_vertical, symbol Connector_Generic:Conn_01x01
- added J6: Inverter_Conn, HeavyDuty:keystone_m3_screw_terminal_vertical, symbol Connector_Generic:Conn_01x01
Connections:
- net GND_HP: now also GND_Conn1.1, J14.1 (Pin_1)
- net at R8.1: now also J6.1 (Pin_1)
- net at R5.1: now also J15.1 (Pin_1)
