File: electronics/high_power.kicad_sch (KiCad schematic)
At the start: 34 parts, among them J12 Conn_01x01, J23 Conn_01x01, J24 Conn_01x01, J4 Conn_01x01, J6 GND_Busbar, J8 Conn_01x01, Q2 AON6407-HXZ, U11 INA3221

Commit message: nerd weekend update
Other:
- added sheet blown_fuse_detection (blown_fuse_detection.kicad_sch)
Changed lines of the file:
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@@
+		)
+	)
+	(sheet
+		(at 139.7 109.22)
+		(size 25.4 17.78)
+		(fields_autoplaced yes)
+		(stroke
+			(width 0.1524)
+			(type solid)
+		)
+		(fill
+			(color 0 0 0 0.0000)
+		)
+		(property "Sheetname" "blown_fuse_detection"
+			(at 139.7 108.5084 0)
+			(effects
+				(font
+					(size 1.27 1.27)
+				)
+				(justify left bottom)
+			)
+		)
+		(property "Sheetfile" "blown_fuse_detection.kicad_sch"
+			(at 139.7 127.5846 0)
+			(effects
+				(font
+					(size 1.27 1.27)
+				)
+				(justify left top)
+			)
+		)
+		(instances
+			(project "electronics"
+				(path "/eeb1234c-eae0-4ac6-a30d-2a978d66d889/da888cb1-ed89-4b09-bf89-340f462f0940"
+					(page "15")
+				)
+			)
 		)
 	)

Commit message: start to create BOM and finalising symbol fields
Parts:
- removed Battery1: ~, HeavyDuty:small_busbar-15mm, symbol HeavyDuty:BusBarConn
- removed Inverter1: ~, HeavyDuty:high_current_pad, symbol HeavyDuty:BusBarConn
- removed J6: GND_Busbar, HeavyDuty:small_busbar-15mm, symbol HeavyDuty:BusBarConn
- removed Q2: AON6407-HXZ, Package_TO_SOT_SMD:SOT-23, symbol Transistor_FET:BSS83P
- added D12: D_Schottky_AKA, Package_TO_SOT_SMD:TO-252-2, symbol Device:D_Schottky_AKA
- added D22: D_Schottky, Diode_THT:D_DO-15_P3.81mm_Vertical_AnodeUp, symbol Device:D_Schottky
- added GND_Conn1: ~, HeavyDuty:small_busbar-15mm, symbol HeavyDuty:BusBarConn
- added J14, J25, J29, J30, J31: Conn_GND, HeavyDuty:keystone_m3_screw_terminal_vertical, symbol Connector_Generic:Conn_01x01
- added J15: Battery_Conn, HeavyDuty:keystone_m3_screw_terminal_vertical, symbol Connector_Generic:Conn_01x01
- added J6: Inverter_Conn, HeavyDuty:keystone_m3_screw_terminal_vertical, symbol Connector_Generic:Conn_01x01
- C5, C6, C7, C8: footprint Capacitor_SMD:C_0805_2012Metric_Pad1.18x1.45mm_HandSolder -> Capacitor_SMD:C_0805_2012Metric
- R10, R11, R12, R13, R7, R9: footprint Resistor_SMD:R_0805_2012Metric_Pad1.20x1.40mm_HandSolder -> Resistor_SMD:R_0805_2012Metric
- R14, R15: footprint Resistor_SMD:R_1206_3216Metric_Pad1.30x1.75mm_HandSolder -> Resistor_SMD:R_0805_2012Metric
Connections:
- net GND_HP: now also GND_Conn1.1, J14.1 (Pin_1), J25.1 (Pin_1), J29.1 (Pin_1), J30.1 (Pin_1), J31.1 (Pin_1)
- net at R8.1: now also J6.1 (Pin_1)
- net at R5.1: now also J15.1 (Pin_1)
- net V_Bat renamed +12V_HP
- net +12V_HP: now also D12.1 (A), D12.3 (A), D22.2 (A)
- new net +12V: D12.2 (K), D22.1 (K)
Other:
- removed sheet blown_fuse_detection
