File: electronics/_autosave-option_2.kicad_sch (KiCad schematic)
At the start: 11 parts, among them Q6 Q_PMOS_GSD, U19 LM339_4ch, U20 LM339_4ch, U5 ULN2801A

Commit message: start to do proper layout
Connections:
- net probe is gone; now on net probe_1: Q6.1 (G), R27.1
- net +3V3: now also Q6.2 (S); no longer Q6.3 (D)
- net MCU_PIN: now also Q6.3 (D); no longer Q6.2 (S)
Other:
- moved on the sheet: R27, R33
