File: electronics/electronics.kicad_pcb (KiCad board)
At the start: 2 copper layers, 214.5 x 134.8 mm, 123 parts, among them J1 rgb_led_conn, J12 Conn_01x01, J16 Conn_01x02, J17 Conn_01x03, J18 Conn_01x03, J2 CAN, J20 water_sensor_conn, J21 Conn_01x02, J22 Conn_01x02, J23 Conn_01x01, J24 Conn_01x01, J25 Conn_01x08, J4 Conn_01x01, J5 DB12, J6 GND_Busbar, J7 Conn_01x02, J8 Conn_01x01, J9 water_sensor_conn, Q1 Q_PMOS_GDS, Q2 AON6407-HXZ, Q3 N-MOS, Q4 N-MOS, Q5 N-MOS, SW1 SW_Push, SW2 SW_Push, SW3 SW_Push, SW4 SW_Push, SW5 SW_Push, U1 AZ1117-ADJ, U10 BTS7006, U11 INA3221, U13 CNY17-1, U15 TCA9555PWR, U16 ULN2003, U17 H11AA1, U2 AZ1117-ADJ, U3 TJA1051T-3, U4 ESP32-S3-MINI-1U, U6 BTS7006, U7 BTS7006, U8 BTS7006, U9 BTS7006

Commit message: from dell
Parts:
- removed Battery1: ~, HeavyDuty:small_busbar-15mm
- removed Inverter1: ~, HeavyDuty:high_current_pad
- removed J16: Conn_01x02, TerminalBlock:TerminalBlock_Xinya_XY308-2.54-2P_1x02_P2.54mm_Horizontal
- removed J20: water_sensor_conn, TerminalBlock:TerminalBlock_Xinya_XY308-2.54-5P_1x05_P2.54mm_Horizontal
- removed Q1: Q_PMOS_GDS, Package_TO_SOT_SMD:SOT-23_Handsoldering
- removed Q2: AON6407-HXZ, Package_TO_SOT_SMD:SOT-23
- removed R17: 1k, Resistor_SMD:R_0805_2012Metric_Pad1.20x1.40mm_HandSolder
- removed R26, R28, R29, R30, R31, R32: 4.7k, Resistor_SMD:R_0805_2012Metric_Pad1.20x1.40mm_HandSolder
- removed U16: ULN2003, Package_SO:SO-16_3.9x9.9mm_P1.27mm
- added C10: 22uF, Capacitor_SMD:C_0805_2012Metric_Pad1.18x1.45mm_HandSolder, F.Cu at (343.7, 112.0)
- added D12: ESD Diode 5V, Diode_SMD:Nexperia_DSN1608-2_1.6x0.8mm, F.Cu at (341.3, 97.5)
- added D13: LED, LED_SMD:LED_1812_4532Metric_Pad1.30x3.40mm_HandSolder, F.Cu at (337.6, 104.1)
- added D14: LED, LED_SMD:LED_1812_4532Metric_Pad1.30x3.40mm_HandSolder, F.Cu at (337.6, 109.2)
- added D15: D_Schottky, Diode_SMD:D_SMB, F.Cu at (338.1, 89.0)
- added D23: SMF5, Diode_SMD:D_SMF, F.Cu at (336.9, 98.0)
- added D24: SMAJ18CA, Diode_SMD:D_SMA, F.Cu at (338.0, 94.0)
- added GND_Conn1: ~, HeavyDuty:small_busbar-15mm, F.Cu at (154.2, 70.2)
- added J10: Conn_01x02, TerminalBlock:TerminalBlock_Xinya_XY308-2.54-2P_1x02_P2.54mm_Horizontal, F.Cu at (115.7, 115.2)
- added J13: water_sensor_conn, TerminalBlock:TerminalBlock_Xinya_XY308-2.54-5P_1x05_P2.54mm_Horizontal, F.Cu at (123.4, 115.2)
- added J14: Conn_GND, HeavyDuty:keystone_m3_screw_terminal_vertical, F.Cu at (153.5, 25.0)
- added J15: Battery_Conn, HeavyDuty:keystone_m3_screw_terminal_vertical, F.Cu at (54.8, 25.5)
- added J3: Conn_01x08, TerminalBlock:TerminalBlock_Xinya_XY308-2.54-8P_1x08_P2.54mm_Horizontal, F.Cu at (145.1, 50.0)
- added R16: 1M, Resistor_SMD:R_0805_2012Metric_Pad1.20x1.40mm_HandSolder, B.Cu at (132.8, 103.8)
- added R27: 4k7, Resistor_SMD:R_0805_2012Metric_Pad1.20x1.40mm_HandSolder, F.Cu at (343.6, 103.1)
- added R33: 475, Resistor_SMD:R_0805_2012Metric_Pad1.20x1.40mm_HandSolder, F.Cu at (343.6, 106.0)
- added R34: 1k, Resistor_SMD:R_0805_2012Metric_Pad1.20x1.40mm_HandSolder, F.Cu at (343.6, 109.0)
- added R35: 100k, Resistor_SMD:R_0805_2012Metric_Pad1.20x1.40mm_HandSolder, B.Cu at (132.8, 106.0)
- added R36: 100k, Resistor_SMD:R_0805_2012Metric_Pad1.20x1.40mm_HandSolder, B.Cu at (132.8, 108.2)
- added R37: 1M, Resistor_SMD:R_0805_2012Metric_Pad1.20x1.40mm_HandSolder, B.Cu at (116.5, 103.2)
- added R38: 1M, Resistor_SMD:R_0805_2012Metric_Pad1.20x1.40mm_HandSolder, B.Cu at (116.5, 105.5)
- added R39: 1M, Resistor_SMD:R_0805_2012Metric_Pad1.20x1.40mm_HandSolder, B.Cu at (132.8, 101.5)
- added U20: LM339_4ch, Package_SO:HTSSOP-14-1EP_4.4x5mm_P0.65mm_EP3.4x5mm_Mask3x3.1mm, B.Cu at (124.0, 104.5)
- added U21: LM339_4ch, Package_SO:HTSSOP-14-1EP_4.4x5mm_P0.65mm_EP3.4x5mm_Mask3x3.1mm, B.Cu at (122.5, 95.5)
- added U5: ESP32-S3-MINI-1, RF_Module:ESP32-S2-MINI-1U, B.Cu at (77.7, 90.0)
- D1: value D -> LED; footprint Diode_SMD:D_1210_3225Metric_Pad1.42x2.65mm_HandSolder -> LED_SMD:LED_1812_4532Metric_Pad1.30x3.40mm_HandSolder
- J6: value GND_Busbar -> Inverter_Conn; footprint HeavyDuty:small_busbar-15mm -> HeavyDuty:keystone_m3_screw_terminal_vertical
- U10, U6, U7, U8, U9: moved to F.Cu
- U4: value ESP32-S3-MINI-1U -> LM339_4ch; footprint RF_Module:ESP32-S2-MINI-1U -> Package_SO:HTSSOP-14-1EP_4.4x5mm_P0.65mm_EP3.4x5mm_Mask3x3.1mm; moved to F.Cu
- moved U4 242.5 mm to (319.1, 113.8), turned to 0 degrees
- moved D17 204.4 mm to (27.2, 154.2)
- moved R14 202.9 mm to (270.8, 80.0)
- moved R15 202.9 mm to (270.7, 83.0)
- moved D21 191.8 mm to (40.0, 154.5)
- moved D3 191.5 mm to (28.8, 130.0)
- moved D4 191.5 mm to (28.8, 135.5)
- moved D5 191.5 mm to (28.8, 141.0)
- moved D6 191.5 mm to (28.8, 146.5)
- moved SW1 179.3 mm to (27.5, 164.0), turned to 90 degrees
- moved D20 179.0 mm to (53.5, 153.2), turned to -90 degrees
- moved D11 168.9 mm to (47.9, 143.6)
- moved D8 168.9 mm to (47.9, 128.3)
- moved D10 168.9 mm to (47.9, 138.5)
- moved D9 168.9 mm to (47.9, 133.4)
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Connections:
- C1 pad 1: /central_control_unit/12V_MCU -> Net-(D15-K)
- C2 pad 2: /central_control_unit/12V_MCU -> Net-(D15-K)
- C9 pad 1: /central_control_unit/230VAC/AC_DETECT -> /central_control_unit/relay_out
- D1 pad 1: /central_control_unit/12V_MCU -> GND_LP
- D1 pad 2: V_Bat -> Net-(D1-A)
- F3 pad 1: V_Bat -> +12V
- F5 pad 1: V_Bat -> +12V
- J6 pad 1: GND_HP -> Net-(J6-Pin_1)
- R22 pad 1: /central_control_unit/230VAC/RELAY_IN -> /central_control_unit/ac_detect
- R25 pad 2: /central_control_unit/230VAC/AC_DETECT -> /central_control_unit/relay_out
- R5 pad 4: V_Bat -> +12V
- R6 pad 4: V_Bat -> +12V
- R8 pad 1: Net-(Inverter1-Pad1) -> Net-(J6-Pin_1)
- R8 pad 4: V_Bat -> +12V
- U1 pad 3: /central_control_unit/12V_MCU -> Net-(D15-K)
- U15 pad 1: Net-(U15-~{INT}) -> unconnected-(U15-~{INT}-Pad1)
- U15 pad 10: /central_control_unit/digital_switching/CH1_IN -> /central_control_unit/relay_out
- U15 pad 11: /central_control_unit/digital_switching/CH1_DEN -> unconnected-(U15-P07-Pad11)
- U15 pad 12: GND_LP -> unconnected-(U15-GND-Pad12)
- U15 pad 13: /central_control_unit/digital_switching/CH2_IN -> unconnected-(U15-P10-Pad13)
- U15 pad 14: /central_control_unit/digital_switching/CH2_DEN -> unconnected-(U15-P11-Pad14)
- U15 pad 15: /central_control_unit/digital_switching/CH3_IN -> unconnected-(U15-P12-Pad15)
- U15 pad 16: /central_control_unit/digital_switching/CH3_DEN -> unconnected-(U15-P13-Pad16)
- U15 pad 17: /central_control_unit/digital_switching/CH4_IN -> unconnected-(U15-P14-Pad17)
- U15 pad 18: /central_control_unit/digital_switching/CH4_DEN -> unconnected-(U15-P15-Pad18)
- U15 pad 19: /central_control_unit/digital_switching/CH5_IN -> unconnected-(U15-P16-Pad19)
- U15 pad 2: GND_LP -> unconnected-(U15-A1-Pad2)
- U15 pad 20: /central_control_unit/digital_switching/CH5_DEN -> unconnected-(U15-P17-Pad20)
- U15 pad 21: GND_LP -> unconnected-(U15-A0-Pad21)
- U15 pad 22: /central_control_unit/SCL -> unconnected-(U15-SCL-Pad22)
- U15 pad 23: /central_control_unit/SDA -> unconnected-(U15-SDA-Pad23)
- U15 pad 24: +3.3V -> unconnected-(U15-VCC-Pad24)
- U15 pad 3: GND_LP -> unconnected-(U15-A2-Pad3)
- U15 pad 4: /central_control_unit/water_sensors_logic/WS_ENABLE -> /central_control_unit/water_sensors_logic/WS_LVL_25%
- U15 pad 5: /central_control_unit/water_sensors_logic/WS_LVL_25% -> /central_control_unit/water_sensors_logic/WS_LVL_50%
- U15 pad 6: /central_control_unit/water_sensors_logic/WS_LVL_50% -> /central_control_unit/water_sensors_logic/WS_LVL_75%
- U15 pad 7: /central_control_unit/water_sensors_logic/WS_LVL_75% -> /central_control_unit/water_sensors_logic/WS_LVL_100%
- U15 pad 8: /central_control_unit/water_sensors_logic/WS_LVL_100% -> /central_control_unit/water_sensors_logic/GREY_WATER_FULL
- U15 pad 9: /central_control_unit/water_sensors_logic/GREY_WATER_FULL -> /central_control_unit/ac_detect
- U17 pad 5: /central_control_unit/230VAC/AC_DETECT -> /central_control_unit/relay_out
- U2 pad 3: /central_control_unit/12V_MCU -> Net-(D15-K)
- U3 pad 1: /central_control_unit/CAN/CAN_TX -> /central_control_unit/can_tx
- U3 pad 4: /central_control_unit/CAN/CAN_RX -> /central_control_unit/can_rx
- U4 pad 1: GND_LP -> BTN2_INTR
- U4 pad 10: /central_control_unit/SDA -> unconnected-(U4-IN4--Pad10)
- U4 pad 11: /central_control_unit/SCL -> unconnected-(U4-IN4+-Pad11)
- U4 pad 13: unconnected-(U4-IO9-Pad13) -> BTN4_INTR
- U4 pad 14: unconnected-(U4-IO10-Pad14) -> BTN3_INTR
- U4 pad 15: /central_control_unit/230VAC/RELAY_IN -> (no net)
- U4 pad 2: GND_LP -> BTN1_INTR
- U4 pad 3: +3.3V -> unconnected-(U4-Vcc-Pad3)
- U4 pad 4: /central_control_unit/strap pin -> unconnected-(U4-IN1--Pad4)
Other:
- board size 214.5 x 134.8 mm -> 150 x 153.5 mm

Commit message: capacitors added. universal dc/dc converters
Parts:
- removed D23: SMF5, Diode_SMD:D_SMF
- removed D24: SMAJ18CA, Diode_SMD:D_SMA
- removed FB2: FerriteBead 47 Ohm, Inductor_SMD:L_Walsin_WLFM201609x
- removed Q5: N-MOS, Package_TO_SOT_SMD:SOT-23
- removed U2: AZ1117-ADJ, Package_TO_SOT_SMD:SOT-223-3_TabPin2
- removed U20, U21: LM339_4ch, Package_SO:HTSSOP-14-1EP_4.4x5mm_P0.65mm_EP3.4x5mm_Mask3x3.1mm
- added C10: 22uF, Capacitor_SMD:C_0805_2012Metric, B.Cu at (67.5, 79.5)
- added C11: 100nF, Capacitor_SMD:C_0805_2012Metric, B.Cu at (84.5, 101.0)
- added C12: 100nF, Capacitor_SMD:C_0805_2012Metric, B.Cu at (89.5, 109.0)
- added C13: C_Polarized, Capacitor_THT:CP_Radial_D5.0mm_P2.50mm, F.Cu at (169.0, 78.8)
- added C14: C, Capacitor_SMD:C_0805_2012Metric, B.Cu at (172.7, 111.2)
- added C15: 1uF, Capacitor_SMD:C_0805_2012Metric, B.Cu at (95.5, 93.0)
- added C16: C_Polarized, Capacitor_THT:CP_Radial_D5.0mm_P2.50mm, F.Cu at (100.0, 105.0)
- added C17: 10uF, Capacitor_SMD:C_0805_2012Metric, F.Cu at (54.5, 223.0)
- added C18: 10uF, Capacitor_SMD:C_0805_2012Metric, F.Cu at (54.5, 226.0)
- added C19: 10uF, Capacitor_SMD:C_0805_2012Metric, F.Cu at (54.5, 229.0)
- added C20: 10uF, Capacitor_SMD:C_0805_2012Metric, F.Cu at (54.5, 232.0)
- added C21: 10uF, Capacitor_SMD:C_0805_2012Metric, F.Cu at (54.5, 235.0)
- added C22: C_Polarized, Capacitor_THT:CP_Radial_D5.0mm_P2.50mm, F.Cu at (81.9, 221.4)
- added C23: C_Polarized, Capacitor_THT:CP_Radial_D5.0mm_P2.50mm, F.Cu at (81.4, 227.9)
- added C24: C_Polarized, Capacitor_THT:CP_Radial_D5.0mm_P2.50mm, F.Cu at (81.9, 235.9)
- added C25: 10uF, Capacitor_SMD:C_0805_2012Metric, B.Cu at (89.5, 104.0)
- added C26: C_Polarized, Capacitor_THT:CP_Radial_D5.0mm_P2.50mm, F.Cu at (93.8, 105.0)
- added C27: 100nF, Capacitor_SMD:C_0805_2012Metric, B.Cu at (89.5, 106.5)
- added C28: C_Polarized, Capacitor_THT:CP_Radial_D5.0mm_P2.50mm, F.Cu at (43.5, 98.2)
- added C29: C_Polarized, Capacitor_THT:CP_Radial_D5.0mm_P2.50mm, F.Cu at (67.5, 98.5)
- added C30: C_Polarized, Capacitor_THT:CP_Radial_D5.0mm_P2.50mm, F.Cu at (51.0, 98.2)
- added C31: C_Polarized, Capacitor_THT:CP_Radial_D5.0mm_P2.50mm, F.Cu at (36.5, 98.2)
- added C32: C_Polarized, Capacitor_THT:CP_Radial_D5.0mm_P2.50mm, F.Cu at (59.0, 98.5)
- added C33: C_Polarized, Capacitor_THT:CP_Radial_D5.0mm_P2.50mm, F.Cu at (114.0, 109.5)
- added D22: D_Schottky, Diode_THT:D_DO-15_P3.81mm_Vertical_AnodeUp, F.Cu at (131.8, 76.7)
- added F6: 5A, HeavyDuty:ATO_fuse_holder, F.Cu at (132.0, 46.1)
- added FB1: FerriteBead 47 Ohm, Inductor_SMD:L_Walsin_WLFM201609x, F.Cu at (185.0, 75.5)
- added J16: USB_C_Receptacle_USB2.0_16P, Connector_USB:USB_C_Receptacle_JAE_DX07S016JA1R1500, B.Cu at (71.5, 116.0)
- added J20: leds_ch2, TerminalBlock:TerminalBlock_Xinya_XY308-2.54-3P_1x03_P2.54mm_Horizontal, F.Cu at (160.0, 106.8)
- added J26: leds_ch3, TerminalBlock:TerminalBlock_Xinya_XY308-2.54-3P_1x03_P2.54mm_Horizontal, F.Cu at (170.5, 106.8)
- added J27: leds_ch4, TerminalBlock:TerminalBlock_Xinya_XY308-2.54-3P_1x03_P2.54mm_Horizontal, F.Cu at (170.5, 116.0)
- added J28: Conn_01x08, TerminalBlock:TerminalBlock_Xinya_XY308-2.54-8P_1x08_P2.54mm_Horizontal, F.Cu at (60.1, 220.4)
- added J29: Conn_GND, HeavyDuty:keystone_m3_screw_terminal_vertical, F.Cu at (187.7, 25.0)
- added J30: Conn_GND, HeavyDuty:keystone_m3_screw_terminal_vertical, F.Cu at (173.9, 25.0)
- added J31: Conn_GND, HeavyDuty:keystone_m3_screw_terminal_vertical, F.Cu at (160.1, 25.0)
- added NT1: NetTie_2, NetTie:NetTie-2_THT_Pad1.0mm, F.Cu at (137.7, 82.5)
- added Q1: Q_NMOS_DGS, Package_TO_SOT_SMD:SOT-323_SC-70, B.Cu at (118.5, 78.0)
- added Q2: Q_PMOS_DGS, Package_TO_SOT_SMD:SOT-323_SC-70, B.Cu at (113.7, 78.0)
- added R17: 120, Resistor_SMD:R_0805_2012Metric, B.Cu at (79.5, 107.0)
- added R26: 100k, Resistor_SMD:R_0805_2012Metric, B.Cu at (150.6, 100.0)
- added R28: 1M, Resistor_SMD:R_0805_2012Metric, B.Cu at (150.6, 95.0)
- added R29: 1M, Resistor_SMD:R_0805_2012Metric, B.Cu at (150.6, 102.5)
- added R30: 1M, Resistor_SMD:R_0805_2012Metric, B.Cu at (137.6, 99.5)
- added R31: 1M, Resistor_SMD:R_0805_2012Metric, B.Cu at (137.6, 96.5)
- added R32: 10k, Resistor_SMD:R_0805_2012Metric, B.Cu at (95.6, 95.5)
- added SW6: SW_DIP_x01, Connector_PinHeader_1.00mm:PinHeader_1x02_P1.00mm_Vertical, F.Cu at (79.0, 116.5)
- added SW7: RST_BTN, Button_Switch_THT:SW_PUSH_6mm_H4.3mm, F.Cu at (132.0, 104.7)
- added SW8: FLASH_BTN, Button_Switch_THT:SW_PUSH_6mm_H4.3mm, F.Cu at (132.0, 113.5)
- added U14: LM339_4ch, Package_SO:SOIC-14_3.9x8.7mm_P1.27mm, B.Cu at (144.2, 95.4)
- added U16: ~, HeavyDuty:generic_dcdc, F.Cu at (167.8, 60.8)
- added U18: ~, HeavyDuty:mini360, F.Cu at (115.0, 89.0)
- added U19: ESP32-S3-MINI-1, PCM_Espressif:ESP32-S3-MINI-1U, B.Cu at (78.8, 87.7)
- C1: value 10uF -> C_Polarized; footprint Capacitor_SMD:C_0805_2012Metric_Pad1.18x1.45mm_HandSolder -> Capacitor_THT:CP_Radial_D5.0mm_P2.50mm; moved to F.Cu
- C10: moved to B.Cu
- C2: value 10uF -> C; footprint Capacitor_SMD:C_0805_2012Metric_Pad1.18x1.45mm_HandSolder -> Capacitor_SMD:C_0805_2012Metric
- C3: value 22uF -> C_Polarized; footprint Capacitor_SMD:C_0805_2012Metric_Pad1.18x1.45mm_HandSolder -> Capacitor_THT:CP_Radial_D5.0mm_P2.50mm; moved to F.Cu
- C4: value 22uF -> C; footprint Capacitor_SMD:C_0805_2012Metric_Pad1.18x1.45mm_HandSolder -> Capacitor_SMD:C_0805_2012Metric
- C5, C6, C7, C8, C9: footprint Capacitor_SMD:C_0805_2012Metric_Pad1.18x1.45mm_HandSolder -> Capacitor_SMD:C_0805_2012Metric
- D1: footprint LED_SMD:LED_1812_4532Metric_Pad1.30x3.40mm_HandSolder -> LED_SMD:LED_1206_3216Metric; moved to F.Cu
- D10, D11, D16, D17, D18, D19, D20, D21, D3, D4, D5, D6, D7, D8, D9: footprint LED_SMD:LED_WS2812B-Mini_PLCC4_3.5x3.5mm -> LED_SMD:LED_WS2812B_PLCC4_5.0x5.0mm_P3.2mm
- D12: value ESD Diode 5V -> D_Schottky_AKA; footprint Diode_SMD:Nexperia_DSN1608-2_1.6x0.8mm -> Package_TO_SOT_SMD:TO-252-2; moved to B.Cu
- D13, D14: footprint LED_SMD:LED_1812_4532Metric_Pad1.30x3.40mm_HandSolder -> LED_SMD:LED_1206_3216Metric
- D15: footprint Diode_SMD:D_SMB -> Diode_SMD:D_SMA; moved to B.Cu
- J1: value rgb_led_conn -> leds_ch1
- J10: value Conn_01x02 -> water_sensor_conn; footprint TerminalBlock:TerminalBlock_Xinya_XY308-2.54-2P_1x02_P2.54mm_Horizontal -> TerminalBlock:TerminalBlock_Xinya_XY308-2.54-5P_1x05_P2.54mm_Horizontal
- J13: value water_sensor_conn -> Conn_01x02; footprint TerminalBlock:TerminalBlock_Xinya_XY308-2.54-5P_1x05_P2.54mm_Horizontal -> TerminalBlock:TerminalBlock_Xinya_XY308-2.54-2P_1x02_P2.54mm_Horizontal
- J25: value Conn_01x08 -> Conn_GND; footprint TerminalBlock:TerminalBlock_Xinya_XY308-2.54-8P_1x08_P2.54mm_Horizontal -> HeavyDuty:keystone_m3_screw_terminal_vertical
- J7: value Conn_01x02 -> grey_water_conn
- Q3: value N-MOS -> Q_PMOS_DGS; footprint Package_TO_SOT_SMD:SOT-23 -> Package_TO_SOT_SMD:SOT-323_SC-70
- Q4: value N-MOS -> Q_NMOS_GDS; footprint Package_TO_SOT_SMD:SOT-23 -> Package_TO_SOT_SMD:TO-252-2
- R1: value 125 -> 10k; footprint Resistor_SMD:R_0805_2012Metric_Pad1.20x1.40mm_HandSolder -> Resistor_SMD:R_0805_2012Metric
- R10, R11, R12, R13, R21, R22, R25, R7, R9, R_DEN1, R_DEN2, R_DEN3, R_DEN4, R_DEN5, R_IN1, R_IN2, R_IN3, R_IN4, R_IN5: footprint Resistor_SMD:R_0805_2012Metric_Pad1.20x1.40mm_HandSolder -> Resistor_SMD:R_0805_2012Metric
- R14, R15: footprint Resistor_SMD:R_1206_3216Metric_Pad1.30x1.75mm_HandSolder -> Resistor_SMD:R_0805_2012Metric
- R16: value 1M -> 100k; footprint Resistor_SMD:R_0805_2012Metric_Pad1.20x1.40mm_HandSolder -> Resistor_SMD:R_0805_2012Metric
- R18, R19, R20: value 4.7k -> 4k7; footprint Resistor_SMD:R_0805_2012Metric_Pad1.20x1.40mm_HandSolder -> Resistor_SMD:R_0805_2012Metric
- R2: value 205 -> 100R; footprint Resistor_SMD:R_0805_2012Metric_Pad1.20x1.40mm_HandSolder -> Resistor_SMD:R_0805_2012Metric
- R27: value 4k7 -> 10k; footprint Resistor_SMD:R_0805_2012Metric_Pad1.20x1.40mm_HandSolder -> Resistor_SMD:R_0805_2012Metric; moved to B.Cu
- R3: value 125 -> 4k7; footprint Resistor_SMD:R_0805_2012Metric_Pad1.20x1.40mm_HandSolder -> Resistor_SMD:R_0805_2012Metric
- R33: value 475 -> 4k7; footprint Resistor_SMD:R_0805_2012Metric_Pad1.20x1.40mm_HandSolder -> Resistor_SMD:R_0805_2012Metric; moved to B.Cu
- R34: value 1k -> 4k7; footprint Resistor_SMD:R_0805_2012Metric_Pad1.20x1.40mm_HandSolder -> Resistor_SMD:R_0805_2012Metric; moved to B.Cu
- R35: value 100k -> 4k7; footprint Resistor_SMD:R_0805_2012Metric_Pad1.20x1.40mm_HandSolder -> Resistor_SMD:R_0805_2012Metric
- R36: value 100k -> 100R; footprint Resistor_SMD:R_0805_2012Metric_Pad1.20x1.40mm_HandSolder -> Resistor_SMD:R_0805_2012Metric
- R37, R38, R39: value 1M -> 10k; footprint Resistor_SMD:R_0805_2012Metric_Pad1.20x1.40mm_HandSolder -> Resistor_SMD:R_0805_2012Metric
- R4: value 370 -> 4k7; footprint Resistor_SMD:R_0805_2012Metric_Pad1.20x1.40mm_HandSolder -> Resistor_SMD:R_0805_2012Metric
- U1: value AZ1117-ADJ -> TLV1117-33
- U4: value LM339_4ch -> ~; footprint Package_SO:HTSSOP-14-1EP_4.4x5mm_P0.65mm_EP3.4x5mm_Mask3x3.1mm -> HeavyDuty:generic_dcdc
- U5: value ESP32-S3-MINI-1 -> LM339_4ch; footprint RF_Module:ESP32-S2-MINI-1U -> Package_SO:SOIC-14_3.9x8.7mm_P1.27mm
- moved D15 263.1 mm to (75.5, 104.0), turned to 180 degrees
- moved C10 257.0 mm to (89.0, 78.0), turned to 180 degrees
- moved R27 248.5 mm to (95.5, 90.5), turned to 180 degrees
- moved U1 230.9 mm to (98.0, 84.5), turned to 0 degrees
- moved D12 216.8 mm to (125.5, 76.9), turned to -90 degrees
- moved C2 181.5 mm to (150.5, 35.5)
- moved U4 176.7 mm to (150.5, 60.8), turned to -90 degrees
- moved J25 174.3 mm to (201.5, 25.0)
- moved R33 172.6 mm to (186.1, 35.5), turned to 180 degrees
- moved C3 170.7 mm to (152.0, 78.8), turned to 180 degrees
- moved R34 170.2 mm to (190.1, 35.5)
- moved R1 167.4 mm to (164.5, 34.0)
- moved R14 163.9 mm to (106.9, 78.0)
- moved R15 163.9 mm to (106.9, 81.0)
- moved R2 158.6 mm to (173.0, 38.5)
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Connections:
- net /central_control_unit/temp_sensors/1-WIRE renamed /central_control_unit/1-Wire
- net Net-(J5-Pin_3) renamed /central_control_unit/digital_switching/CH3_OUT
- C1 pad 1: Net-(D15-K) -> Net-(Q3-S)
- C1 pad 2: GND_LP -> GND_HP
- C2 pad 1: GND_LP -> Net-(Q3-S)
- C2 pad 2: Net-(D15-K) -> GND_HP
- C3 pad 1: Net-(C3-Pad1) -> /central_control_unit/lightning/LEDS_CH12_5V
- C3 pad 2: +3.3V -> /central_control_unit/lightning/leds12_gnd
- C4 pad 1: GND -> /central_control_unit/lightning/LEDS_CH12_5V
- C4 pad 2: +5V -> /central_control_unit/lightning/leds12_gnd
- C9 pad 1: /central_control_unit/relay_out -> /central_control_unit/ac_detect
- D10 pad 1: unconnected-(D10-VDD-Pad1) -> /analog_ui/+5V_UI
- D10 pad 2: unconnected-(D10-DOUT-Pad2) -> Net-(D10-DOUT)
- D10 pad 3: unconnected-(D10-VSS-Pad3) -> /analog_ui/GND_UI
- D10 pad 4: unconnected-(D10-DIN-Pad4) -> Net-(D10-DIN)
- D11 pad 1: unconnected-(D11-VDD-Pad1) -> /analog_ui/+5V_UI
- D11 pad 2: unconnected-(D11-DOUT-Pad2) -> Net-(D11-DOUT)
- D11 pad 3: unconnected-(D11-VSS-Pad3) -> /analog_ui/GND_UI
- D11 pad 4: unconnected-(D11-DIN-Pad4) -> Net-(D10-DOUT)
- D12 pad 1: unconnected-(D12-K-Pad1) -> +12V_HP
- D12 pad 2: unconnected-(D12-A-Pad2) -> +12V
- D15 pad 1: Net-(D15-K) -> /central_control_unit/USB_VBUS
- D15 pad 2: +12V -> /central_control_unit/USB_VIN
- D16 pad 1: unconnected-(D16-VDD-Pad1) -> /analog_ui/+5V_UI
- D16 pad 2: unconnected-(D16-DOUT-Pad2) -> Net-(D16-DOUT)
- D16 pad 3: unconnected-(D16-VSS-Pad3) -> /analog_ui/GND_UI
- D16 pad 4: unconnected-(D16-DIN-Pad4) -> Net-(D16-DIN)
- D17 pad 1: unconnected-(D17-VDD-Pad1) -> /analog_ui/+5V_UI
- D17 pad 2: unconnected-(D17-DOUT-Pad2) -> Net-(D17-DOUT)
- D17 pad 3: unconnected-(D17-VSS-Pad3) -> /analog_ui/GND_UI
- D17 pad 4: unconnected-(D17-DIN-Pad4) -> Net-(D16-DOUT)
- D18 pad 1: unconnected-(D18-VDD-Pad1) -> /analog_ui/+5V_UI
- D18 pad 2: unconnected-(D18-DOUT-Pad2) -> Net-(D18-DOUT)
- D18 pad 3: unconnected-(D18-VSS-Pad3) -> /analog_ui/GND_UI
- D18 pad 4: unconnected-(D18-DIN-Pad4) -> Net-(D17-DOUT)
- D19 pad 1: unconnected-(D19-VDD-Pad1) -> /analog_ui/+5V_UI
- D19 pad 2: unconnected-(D19-DOUT-Pad2) -> Net-(D19-DOUT)
- D19 pad 3: unconnected-(D19-VSS-Pad3) -> /analog_ui/GND_UI
- D19 pad 4: unconnected-(D19-DIN-Pad4) -> Net-(D18-DOUT)
- D20 pad 1: unconnected-(D20-VDD-Pad1) -> /analog_ui/+5V_UI
- D20 pad 2: unconnected-(D20-DOUT-Pad2) -> Net-(D20-DOUT)
- D20 pad 3: unconnected-(D20-VSS-Pad3) -> /analog_ui/GND_UI
- D20 pad 4: unconnected-(D20-DIN-Pad4) -> Net-(D19-DOUT)
- D21 pad 1: unconnected-(D21-VDD-Pad1) -> /analog_ui/+5V_UI
- D21 pad 3: unconnected-(D21-VSS-Pad3) -> /analog_ui/GND_UI
- D21 pad 4: unconnected-(D21-DIN-Pad4) -> Net-(D20-DOUT)
- D3 pad 1: unconnected-(D3-VDD-Pad1) -> /analog_ui/+5V_UI
- D3 pad 2: unconnected-(D3-DOUT-Pad2) -> Net-(D3-DOUT)
- D3 pad 3: unconnected-(D3-VSS-Pad3) -> /analog_ui/GND_UI
- D3 pad 4: unconnected-(D3-DIN-Pad4) -> /analog_ui/LED_DATA_IN
- D4 pad 1: unconnected-(D4-VDD-Pad1) -> /analog_ui/+5V_UI
- D4 pad 2: unconnected-(D4-DOUT-Pad2) -> Net-(D4-DOUT)
- D4 pad 3: unconnected-(D4-VSS-Pad3) -> /analog_ui/GND_UI
- D4 pad 4: unconnected-(D4-DIN-Pad4) -> Net-(D3-DOUT)
- D5 pad 1: unconnected-(D5-VDD-Pad1) -> /analog_ui/+5V_UI
- D5 pad 2: unconnected-(D5-DOUT-Pad2) -> Net-(D5-DOUT)
- D5 pad 3: unconnected-(D5-VSS-Pad3) -> /analog_ui/GND_UI
- D5 pad 4: unconnected-(D5-DIN-Pad4) -> Net-(D4-DOUT)
- D6 pad 1: unconnected-(D6-VDD-Pad1) -> /analog_ui/+5V_UI
- D6 pad 2: unconnected-(D6-DOUT-Pad2) -> Net-(D6-DOUT)
- D6 pad 3: unconnected-(D6-VSS-Pad3) -> /analog_ui/GND_UI
- D6 pad 4: unconnected-(D6-DIN-Pad4) -> Net-(D5-DOUT)
- D7 pad 1: unconnected-(D7-VDD-Pad1) -> /analog_ui/+5V_UI
- D7 pad 2: unconnected-(D7-DOUT-Pad2) -> Net-(D16-DIN)
- D7 pad 3: unconnected-(D7-VSS-Pad3) -> /analog_ui/GND_UI
- D7 pad 4: unconnected-(D7-DIN-Pad4) -> Net-(D11-DOUT)
- D8 pad 1: unconnected-(D8-VDD-Pad1) -> /analog_ui/+5V_UI
- D8 pad 3: unconnected-(D8-VSS-Pad3) -> /analog_ui/GND_UI
- D8 pad 4: unconnected-(D8-DIN-Pad4) -> Net-(D6-DOUT)
- D9 pad 1: unconnected-(D9-VDD-Pad1) -> /analog_ui/+5V_UI
- D9 pad 2: unconnected-(D9-DOUT-Pad2) -> Net-(D10-DIN)
- D9 pad 3: unconnected-(D9-VSS-Pad3) -> /analog_ui/GND_UI
- F3 pad 1: +12V -> +12V_HP
- F5 pad 1: +12V -> +12V_HP
- J1 pad 1: Net-(J1-Pin_1) -> /central_control_unit/lightning/LEDS_CH12_5V
- J1 pad 2: Net-(J1-Pin_2) -> /central_control_unit/LED_CH1
- J1 pad 3: Net-(J1-Pin_3) -> /central_control_unit/lightning/leds12_gnd
- J10 pad 2: /central_control_unit/water_sensors_logic/grey_water_probe -> /central_control_unit/water_sensors_logic/probe_4
- J13 pad 2: /central_control_unit/water_sensors_logic/probe_1 -> /central_control_unit/water_sensors_logic/grey_water_probe
- J17 pad 3: GND -> GND_LP
- J18 pad 3: GND -> GND_LP
- J2 pad 2: /central_control_unit/CAN/CAN_L -> /central_control_unit/can_term_r_dip_2
- J25 pad 1: unconnected-(J25-Pin_1-Pad1) -> GND_HP
- J3 pad 1: /central_control_unit/analog_ui_control/+5V_OUT -> +5V
- J3 pad 2: /central_control_unit/analog_ui_control/GND_OUT -> GND_LP
- J3 pad 3: /central_control_unit/analog_ui_control/LED_DATA_IN -> /central_control_unit/analog_ui_rmt_led
- J3 pad 4: /central_control_unit/analog_ui_control/BTN_1_IN -> /central_control_unit/btn_1
- J3 pad 5: /central_control_unit/analog_ui_control/BTN_2_IN -> /central_control_unit/btn_2
- J3 pad 6: /central_control_unit/analog_ui_control/BTN_3_IN -> /central_control_unit/btn_3
- J3 pad 7: /central_control_unit/analog_ui_control/BTN_4_IN -> /central_control_unit/btn_4
- J3 pad 8: /central_control_unit/analog_ui_control/BTN_5_IN -> /central_control_unit/btn_5
- J5 pad 1: Net-(J5-Pin_1) -> /central_control_unit/digital_switching/CH5_OUT
- J5 pad 2: Net-(J5-Pin_2) -> /central_control_unit/digital_switching/CH4_OUT
- J5 pad 4: Net-(J5-Pin_4) -> /central_control_unit/digital_switching/CH2_OUT
- J5 pad 5: Net-(J5-Pin_5) -> /central_control_unit/digital_switching/CH1_OUT
- Q3 pad 1: /central_control_unit/LED_R -> Net-(Q3-D)
- Q3 pad 2: Net-(J1-Pin_1) -> Net-(Q3-G)
- Q3 pad 3: GND_HP -> Net-(Q3-S)
- Q4 pad 1: /central_control_unit/LED_B -> Net-(Q3-D)
- Q4 pad 2: Net-(J1-Pin_3) -> Net-(Q4-D)
- R1 pad 1: +3.3V -> Net-(Q3-D)
- R1 pad 2: Net-(U1-ADJ) -> GND_HP
- R16 pad 1: +3V3 -> /central_control_unit/water_sensors_logic/ws_vref
- R16 pad 2: /central_control_unit/water_sensors_logic/probe_3 -> +3V3
- R18 pad 1: /central_control_unit/LED_R -> Net-(R18-Pad1)
- R18 pad 2: GND_HP -> +5V
- R19 pad 1: /central_control_unit/LED_G -> Net-(J16-CC1)
- R19 pad 2: GND_HP -> GND_LP
- R2 pad 1: Net-(U1-ADJ) -> /central_control_unit/led_en
- R2 pad 2: GND_LP -> Net-(Q3-G)
- R20 pad 1: /central_control_unit/LED_B -> Net-(J16-CC2)
- R20 pad 2: GND_HP -> GND_LP
- R22 pad 1: /central_control_unit/ac_detect -> /central_control_unit/relay_out
- R25 pad 2: /central_control_unit/relay_out -> /central_control_unit/ac_detect
- R27 pad 1: Net-(D1-A) -> +3.3V
- R27 pad 2: +12V -> /central_control_unit/ESP_EN
- R3 pad 1: +5V -> Net-(D14-A)
- R3 pad 2: Net-(U2-ADJ) -> Net-(R18-Pad1)
- R33 pad 1: Net-(D13-A) -> Net-(R33-Pad1)
- R33 pad 2: +3.3V -> +12V
- R34 pad 1: Net-(D14-A) -> Net-(R33-Pad1)
- R34 pad 2: +5V -> Net-(R34-Pad2)
- R35 pad 1: /central_control_unit/water_sensors_logic/ws_vref -> Net-(D1-A)
- R35 pad 2: +3V3 -> Net-(R34-Pad2)
- R36 pad 1: GND -> Net-(Q1-G)
- R36 pad 2: /central_control_unit/water_sensors_logic/ws_vref -> /central_control_unit/USB_VBUS
- R37 pad 1: +3V3 -> Net-(Q1-G)
- R37 pad 2: /central_control_unit/water_sensors_logic/probe_2 -> GND_LP
- R38 pad 1: +3V3 -> +12V
- R38 pad 2: /central_control_unit/water_sensors_logic/probe_1 -> Net-(Q1-D)
- R39 pad 1: +3V3 -> Net-(Q3-G)
- R39 pad 2: /central_control_unit/water_sensors_logic/probe_4 -> Net-(Q3-S)
- R4 pad 1: Net-(U2-ADJ) -> Net-(D13-A)
- R4 pad 2: GND_LP -> +3.3V
- R5 pad 4: +12V -> +12V_HP
- R6 pad 4: +12V -> +12V_HP
- R8 pad 4: +12V -> +12V_HP
- R_DEN1 pad 1: /central_control_unit/digital_switching/CH1_DEN -> /central_control_unit/ch1_den
- R_DEN2 pad 1: /central_control_unit/digital_switching/CH2_DEN -> /central_control_unit/ch2_den
- R_DEN3 pad 1: /central_control_unit/digital_switching/CH3_DEN -> /central_control_unit/ch3_den
- R_DEN4 pad 1: /central_control_unit/digital_switching/CH4_DEN -> /central_control_unit/ch4_den
- R_DEN5 pad 1: /central_control_unit/digital_switching/CH5_DEN -> /central_control_unit/ch5_den
- R_IN1 pad 1: /central_control_unit/digital_switching/CH1_IN -> /central_control_unit/ch1_in
- R_IN2 pad 1: /central_control_unit/digital_switching/CH2_IN -> /central_control_unit/ch2_in
- R_IN3 pad 1: /central_control_unit/digital_switching/CH3_IN -> /central_control_unit/ch3_in
- R_IN4 pad 1: /central_control_unit/digital_switching/CH4_IN -> /central_control_unit/ch4_in
- R_IN5 pad 1: /central_control_unit/digital_switching/CH5_IN -> /central_control_unit/ch5_in
- SW1 pad 1: GND_LP -> /analog_ui/GND_UI
- SW1 pad 2: unconnected-(SW1-Pad2) -> /analog_ui/BTN_1_IN
- SW2 pad 1: GND_LP -> /analog_ui/GND_UI
- SW2 pad 2: unconnected-(SW2-Pad2) -> /analog_ui/BTN_2_IN
- SW3 pad 1: GND_LP -> /analog_ui/GND_UI
- SW3 pad 2: unconnected-(SW3-Pad2) -> /analog_ui/BTN_3_IN
- SW4 pad 1: GND_LP -> /analog_ui/GND_UI
- SW4 pad 2: unconnected-(SW4-Pad2) -> /analog_ui/BTN_4_IN
- SW5 pad 1: GND_LP -> /analog_ui/GND_UI
- SW5 pad 2: unconnected-(SW5-Pad2) -> /analog_ui/BTN_5_IN
- U1 pad 1: Net-(U1-ADJ) -> GND_LP
- U1 pad 3: Net-(D15-K) -> +5V
- U10 pad 10: Net-(J5-Pin_5) -> /central_control_unit/digital_switching/CH5_OUT
- U10 pad 12: Net-(J5-Pin_5) -> /central_control_unit/digital_switching/CH5_OUT
- U10 pad 13: Net-(J5-Pin_5) -> /central_control_unit/digital_switching/CH5_OUT
- U10 pad 14: Net-(J5-Pin_5) -> /central_control_unit/digital_switching/CH5_OUT
- U10 pad 15: V_Bat -> +12V_HP
- U10 pad 8: Net-(J5-Pin_5) -> /central_control_unit/digital_switching/CH5_OUT
- U10 pad 9: Net-(J5-Pin_5) -> /central_control_unit/digital_switching/CH5_OUT
- U15 pad 10: /central_control_unit/relay_out -> /central_control_unit/WS_LVL_25
- U15 pad 11: unconnected-(U15-P07-Pad11) -> /central_control_unit/can_sleep
- U15 pad 12: unconnected-(U15-GND-Pad12) -> GND_LP
- U15 pad 13: unconnected-(U15-P10-Pad13) -> /central_control_unit/can_term_r_dip_1
- U15 pad 14: unconnected-(U15-P11-Pad14) -> /central_control_unit/can_term_r_dip_2
- U15 pad 2: unconnected-(U15-A1-Pad2) -> GND_LP
- U15 pad 21: unconnected-(U15-A0-Pad21) -> GND_LP
- U15 pad 22: unconnected-(U15-SCL-Pad22) -> /central_control_unit/SCL
- U15 pad 23: unconnected-(U15-SDA-Pad23) -> /central_control_unit/SDA
- U15 pad 24: unconnected-(U15-VCC-Pad24) -> +3.3V
- U15 pad 3: unconnected-(U15-A2-Pad3) -> GND_LP
- U15 pad 4: /central_control_unit/water_sensors_logic/WS_LVL_25% -> /central_control_unit/relay_out
- U15 pad 5: /central_control_unit/water_sensors_logic/WS_LVL_50% -> /central_control_unit/ac_detect
- U15 pad 6: /central_control_unit/water_sensors_logic/WS_LVL_75% -> /central_control_unit/GREY_FULL
- U15 pad 7: /central_control_unit/water_sensors_logic/WS_LVL_100% -> /central_control_unit/WS_LVL_100
- U15 pad 8: /central_control_unit/water_sensors_logic/GREY_WATER_FULL -> /central_control_unit/WS_LVL_75
- U15 pad 9: /central_control_unit/ac_detect -> /central_control_unit/WS_LVL_50
- U17 pad 5: /central_control_unit/relay_out -> /central_control_unit/ac_detect
- U3 pad 2: GND -> GND_LP
- U3 pad 5: Net-(U3-VIO) -> /central_control_unit/CAN/can_vio
- U3 pad 6: /central_control_unit/CAN/CAN_L -> /central_control_unit/can_term_r_dip_2
- U3 pad 8: /central_control_unit/CAN/CAN_SLEEP -> /central_control_unit/can_sleep
- U4 pad 1: BTN2_INTR -> Net-(Q3-S)
- U4 pad 2: BTN1_INTR -> Net-(Q4-D)
- U4 pad 3: unconnected-(U4-Vcc-Pad3) -> /central_control_unit/lightning/LEDS_CH12_5V
- U4 pad 4: unconnected-(U4-IN1--Pad4) -> /central_control_unit/lightning/leds12_gnd
- U5 pad 1: GND_LP -> unconnected-(U5-OUT2-Pad1)
- U5 pad 12: unconnected-(U5-GPIO8/TOUCH8/ADC1_CH7/SUBSPICS1-Pad12) -> GND_LP
- U5 pad 2: GND_LP -> /central_control_unit/GREY_FULL
- U5 pad 3: +3.3V -> +3V3
- U5 pad 4: unconnected-(U5-GPIO0/BOOT-Pad4) -> /central_control_unit/water_sensors_logic/grey_water_probe
- U5 pad 5: unconnected-(U5-GPIO1/TOUCH1/ADC1_CH0-Pad5) -> /central_control_unit/water_sensors_logic/ws_vref
- U6 pad 10: Net-(J5-Pin_1) -> /central_control_unit/digital_switching/CH1_OUT
- U6 pad 12: Net-(J5-Pin_1) -> /central_control_unit/digital_switching/CH1_OUT
- U6 pad 13: Net-(J5-Pin_1) -> /central_control_unit/digital_switching/CH1_OUT
- U6 pad 14: Net-(J5-Pin_1) -> /central_control_unit/digital_switching/CH1_OUT
- U6 pad 15: V_Bat -> +12V_HP
- U6 pad 8: Net-(J5-Pin_1) -> /central_control_unit/digital_switching/CH1_OUT
- U6 pad 9: Net-(J5-Pin_1) -> /central_control_unit/digital_switching/CH1_OUT
- U7 pad 10: Net-(J5-Pin_2) -> /central_control_unit/digital_switching/CH2_OUT
- U7 pad 12: Net-(J5-Pin_2) -> /central_control_unit/digital_switching/CH2_OUT
- U7 pad 13: Net-(J5-Pin_2) -> /central_control_unit/digital_switching/CH2_OUT
- U7 pad 14: Net-(J5-Pin_2) -> /central_control_unit/digital_switching/CH2_OUT
- U7 pad 15: V_Bat -> +12V_HP
- U7 pad 8: Net-(J5-Pin_2) -> /central_control_unit/digital_switching/CH2_OUT
- U7 pad 9: Net-(J5-Pin_2) -> /central_control_unit/digital_switching/CH2_OUT
- U8 pad 15: V_Bat -> +12V_HP
- U9 pad 10: Net-(J5-Pin_4) -> /central_control_unit/digital_switching/CH4_OUT
- U9 pad 12: Net-(J5-Pin_4) -> /central_control_unit/digital_switching/CH4_OUT
- U9 pad 13: Net-(J5-Pin_4) -> /central_control_unit/digital_switching/CH4_OUT
- U9 pad 14: Net-(J5-Pin_4) -> /central_control_unit/digital_switching/CH4_OUT
- U9 pad 15: V_Bat -> +12V_HP
- U9 pad 8: Net-(J5-Pin_4) -> /central_control_unit/digital_switching/CH4_OUT
- U9 pad 9: Net-(J5-Pin_4) -> /central_control_unit/digital_switching/CH4_OUT
Routing:
- net /central_control_unit/relay_out: track 0.00 -> 70.3 mm
- net /central_control_unit/ac_detect: track 0.00 -> 59.4 mm
- net /central_control_unit/led_en: track 0.00 -> 52.7 mm
- net /central_control_unit/water_sensors_logic/probe_4: track 0.00 -> 33.7 mm
- net /central_control_unit/water_sensors_logic/probe_3: track 0.00 -> 25.7 mm
- net /central_control_unit/water_sensors_logic/probe_1: track 0.00 -> 25.2 mm
- net /central_control_unit/water_sensors_logic/grey_water_probe: track 0.00 -> 24.8 mm, vias 0 -> 1
- net /central_control_unit/water_sensors_logic/probe_2: track 0.00 -> 21.3 mm
- net /central_control_unit/water_sensors_logic/ws_vref: track 0.00 -> 18.3 mm
- net /central_control_unit/WS_LVL_100: track 0.00 -> 17.3 mm
- net /central_control_unit/WS_LVL_75: track 0.00 -> 15.3 mm
- net /central_control_unit/lightning/leds34_gnd: track 0.00 -> 11.1 mm
- net /central_control_unit/WS_LVL_25: track 0.00 -> 4.95 mm
- net /central_control_unit/WS_LVL_50: track 0.00 -> 4.70 mm
- net /central_control_unit/GREY_FULL: track 0.00 -> 2.96 mm
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- added copper zone on B.Cu, net +12V_HP
- added copper zone on F.Cu, net +12V_HP
- added copper zone on B.Cu, net GND_HP
- removed copper zone on B.Cu, net V_Bat
- removed copper zone on F.Cu, net V_Bat
Other:
- board size 150 x 153.5 mm -> 201.6 x 244.9 mm
- board text removed: "RGB_LED logic"
- board text removed: "water_sensor_logic"
