File: electronics/electronics.kicad_pcb (KiCad board)
At the start: 2 copper layers, 100 x 100 mm, 39 parts, among them J1 GND NetTie, J2 CAN Conn, J3 Conn 12V Out 5ch, J4 Conn_01x02, U1 AZ1117-ADJ, U10 BTS7006, U2 AZ1117-ADJ, U3 TJA1051T-3, U4 ESP32-S3-MINI-1U, U5 CD74HC4067SM, U6 BTS7006, U7 BTS7006, U8 BTS7006, U9 BTS7006

Commit message: from Legion
Parts:
- removed BusBar1: ~, HeavyDuty:busbar-20mm
- added Battery1: ~, HeavyDuty:high_current_pad, F.Cu at (41.5, 27.5)
- added C5: 1uF, Capacitor_SMD:C_0805_2012Metric_Pad1.18x1.45mm_HandSolder, B.Cu at (65.0, 46.5)
- added C6: 1uF, Capacitor_SMD:C_0805_2012Metric_Pad1.18x1.45mm_HandSolder, B.Cu at (62.5, 52.5)
- added C7: 1uF, Capacitor_SMD:C_0805_2012Metric_Pad1.18x1.45mm_HandSolder, B.Cu at (69.0, 56.0)
- added C8: 1uF, Capacitor_SMD:C_0805_2012Metric_Pad1.18x1.45mm_HandSolder, B.Cu at (70.0, 47.0)
- added F1: 20A, HeavyDuty:ATO_fuse_holder, F.Cu at (89.5, 49.1)
- added F2: 20A, HeavyDuty:ATO_fuse_holder, F.Cu at (79.5, 49.1)
- added F4: 20A, HeavyDuty:ATO_fuse_holder, F.Cu at (99.5, 49.1)
- added Inverter1: ~, HeavyDuty:high_current_pad, F.Cu at (61.5, 27.5)
- added J11: ~, HeavyDuty:water_sensor_rods, F.Cu at (160.0, 43.5)
- added J5: 12V_BusBar, HeavyDuty:half_busbar-15mm, F.Cu at (45.0, 80.5)
- added J6: GND_Busbar, HeavyDuty:half_busbar-15mm, F.Cu at (115.0, 80.5)
- added J7: Conn_01x02, Connector_Samtec_HPM_THT:Samtec_HPM-02-01-x-S_Straight_1x02_Pitch5.08mm, F.Cu at (158.2, 59.5)
- added J9: water_sensor_conn, TerminalBlock:TerminalBlock_Xinya_XY308-2.54-6P_1x06_P2.54mm_Horizontal, F.Cu at (153.8, 32.5)
- added MH1: MH, MountingHole:MountingHole_3.2mm_M3_ISO7380_Pad_TopBottom, F.Cu at (25.0, 25.0)
- added MH2: MH, MountingHole:MountingHole_3.2mm_M3_ISO7380_Pad_TopBottom, F.Cu at (135.0, 25.0)
- added MH3: MH, MountingHole:MountingHole_3.2mm_M3_ISO7380_Pad_TopBottom, F.Cu at (135.0, 135.0)
- added MH4: MH, MountingHole:MountingHole_3.2mm_M3_ISO7380_Pad_TopBottom, F.Cu at (25.0, 135.0)
- added R10: 10 ohm, Resistor_SMD:R_0805_2012Metric_Pad1.20x1.40mm_HandSolder, B.Cu at (59.5, 51.5)
- added R11: 10 ohm, Resistor_SMD:R_0805_2012Metric_Pad1.20x1.40mm_HandSolder, B.Cu at (59.5, 53.5)
- added R12: 10 ohm, Resistor_SMD:R_0805_2012Metric_Pad1.20x1.40mm_HandSolder, B.Cu at (62.0, 45.5)
- added R13: 10 ohm, Resistor_SMD:R_0805_2012Metric_Pad1.20x1.40mm_HandSolder, B.Cu at (62.0, 47.5)
- added R14: 4.7k, Resistor_SMD:R_1206_3216Metric_Pad1.30x1.75mm_HandSolder, B.Cu at (116.0, 107.0)
- added R15: 4.7k, Resistor_SMD:R_1206_3216Metric_Pad1.30x1.75mm_HandSolder, B.Cu at (116.0, 111.0)
- added R5: 0.001 Ohm 10W, HeavyDuty:MSRSF_shunt_resistor, F.Cu at (43.5, 50.5)
- added R6: 0.003 Ohm 10W, HeavyDuty:MSRSF_shunt_resistor, F.Cu at (71.0, 66.5)
- added R7: 10 ohm, Resistor_SMD:R_0805_2012Metric_Pad1.20x1.40mm_HandSolder, B.Cu at (68.0, 59.0)
- added R8: 0.001 Ohm 10W, HeavyDuty:MSRSF_shunt_resistor, F.Cu at (55.0, 50.5)
- added R9: 10 ohm, Resistor_SMD:R_0805_2012Metric_Pad1.20x1.40mm_HandSolder, B.Cu at (70.0, 59.0)
- added U11: INA3221, Package_DFN_QFN:Texas_RGV0016A_VQFN-16-1EP_4x4mm_P0.65mm_EP2.1x2.1mm, B.Cu at (67.0, 51.5)
- added U12: ~, HeavyDuty:2_water_sensor_rods, F.Cu at (160.8, 68.8)
- C1, C2, C3, C4, C_GND1, C_GND2, C_GND3, C_GND4, C_GND5, D1, J1, R1, R2, R3, R4, R_DEN1, R_DEN2, R_DEN3, R_DEN4, R_DEN5, R_IN1, R_IN2, R_IN3, R_IN4, R_IN5, U1, U10, U2, U3, U4, U5, U6, U7, U8, U9: moved to B.Cu
- J2: value CAN Conn -> Conn_01x02
- J4: value Conn_01x02 -> Chargers_Conn; footprint TerminalBlock_MetzConnect:TerminalBlock_MetzConnect_Type703_RT10N02HGLU_1x02_P9.52mm_Horizontal -> HeavyDuty:3p_terminal
- moved J4 113.9 mm to (89.5, 28.0), turned to 180 degrees
- moved C1 96.6 mm to (155.0, 98.5), turned to 0 degrees
- moved J2 89.7 mm to (152.2, 131.2)
- moved U2 89.4 mm to (151.8, 106.7)
- moved U3 88.7 mm to (151.8, 121.2)
- moved R3 87.4 mm to (150.8, 98.5), turned to 180 degrees
- moved C4 84.6 mm to (150.4, 112.5), turned to 0 degrees
- moved R4 78.6 mm to (146.4, 98.5), turned to 180 degrees
- moved R_DEN5 75.8 mm to (59.5, 110.0)
- moved C_GND1 74.5 mm to (28.9, 128.0), turned to 180 degrees
- moved C_GND2 74.5 mm to (36.4, 128.0), turned to 180 degrees
- moved R_IN5 74.3 mm to (57.6, 110.0)
- moved C_GND3 74.1 mm to (44.4, 128.0), turned to 180 degrees
- moved C_GND4 74.1 mm to (51.4, 128.0), turned to 180 degrees
- moved C_GND5 74.1 mm to (58.4, 128.0), turned to 180 degrees
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Connections:
- net +12V renamed /central_control_unit/12V_MCU
- net +3V3 renamed Net-(U3-VIO)
- net /centra_control_unit/CH1_DIAG renamed /central_control_unit/CH1_DIAG
- net /centra_control_unit/CH1_IN renamed /central_control_unit/CH1_IN
- net /centra_control_unit/CH2_DIAG renamed /central_control_unit/CH2_DIAG
- net /centra_control_unit/CH3_DIAG renamed /central_control_unit/CH3_DIAG
- net /centra_control_unit/DAC_1 renamed /central_control_unit/DAC_1
- net /centra_control_unit/DAC_2 renamed /central_control_unit/DAC_2
- net /centra_control_unit/HP_GND renamed /central_control_unit/HP_GND
- net /centra_control_unit/V_Bat renamed /central_control_unit/V_Bat
- net /centra_control_unit/strap pin renamed /central_control_unit/strap pin
- C3 pad 1: GND -> Net-(C3-Pad1)
- J2 pad 1: /centra_control_unit/CAN_L -> /central_control_unit/CAN_H
- J2 pad 2: /centra_control_unit/CAN_H -> /central_control_unit/CAN_L
- J4 pad 1: +BATT -> Net-(J4-Pin_1)
- J4 pad 2: -BATT -> Net-(J4-Pin_2)
- R4 pad 2: GND -> Net-(R4-Pad2)
- R_DEN1 pad 1: /centra_control_unit/CH1_DIAG_EN -> /central_control_unit/CH1_DIAG_EN
- R_DEN2 pad 1: /centra_control_unit/CH2_DAIG_EN -> /central_control_unit/CH2_DAIG_EN
- R_DEN3 pad 1: /centra_control_unit/CH3_DAIG_EN -> /central_control_unit/CH3_DAIG_EN
- R_DEN4 pad 1: /centra_control_unit/CH4_DAIG_EN -> /central_control_unit/CH4_DAIG_EN
- R_DEN5 pad 1: /centra_control_unit/CH5_DAIG_EN -> /central_control_unit/CH5_DAIG_EN
- R_IN2 pad 1: /centra_control_unit/CH2_IN -> /central_control_unit/CH2_IN
- R_IN3 pad 1: /centra_control_unit/CH3_IN -> /central_control_unit/CH3_IN
- R_IN4 pad 1: /centra_control_unit/CH4_IN -> /central_control_unit/CH4_IN
- R_IN5 pad 1: /centra_control_unit/CH5_IN -> /central_control_unit/CH5_IN
- U10 pad 4: /centra_control_unit/CH4_DIAG -> /central_control_unit/CH5_DIAG
- U3 pad 1: /centra_control_unit/CAN_TX -> /central_control_unit/CAN_TX
- U3 pad 4: /centra_control_unit/CAN_RX -> /central_control_unit/CAN_RX
- U3 pad 6: /centra_control_unit/CAN_L -> /central_control_unit/CAN_L
- U3 pad 7: /centra_control_unit/CAN_H -> /central_control_unit/CAN_H
- U3 pad 8: /centra_control_unit/CAN_SLEEP -> /central_control_unit/CAN_SLEEP
- U4 pad 10: unconnected-(U4-IO6-Pad10) -> /central_control_unit/SDA
- U4 pad 11: unconnected-(U4-IO7-Pad11) -> /central_control_unit/SCL
- U4 pad 12: unconnected-(U4-IO8-Pad12) -> /central_control_unit/CAN_TX
- U4 pad 13: unconnected-(U4-IO9-Pad13) -> /central_control_unit/CAN_RX
- U4 pad 14: /centra_control_unit/CAN_TX -> /central_control_unit/CAN_SLEEP
- U4 pad 15: /centra_control_unit/CAN_RX -> unconnected-(U4-IO11-Pad15)
- U4 pad 16: /centra_control_unit/CAN_SLEEP -> /central_control_unit/MUX_ANALOG_COM
- U4 pad 17: unconnected-(U4-IO13-Pad17) -> /central_control_unit/MUX_S3
- U4 pad 18: unconnected-(U4-IO14-Pad18) -> /central_control_unit/MUX_S2
- U4 pad 19: unconnected-(U4-IO15-Pad19) -> /central_control_unit/MUX_S1
- U4 pad 20: unconnected-(U4-IO16-Pad20) -> /central_control_unit/MUX_S0
- U4 pad 27: unconnected-(U4-IO47-Pad27) -> /central_control_unit/CH1_DIAG_EN
- U4 pad 31: unconnected-(U4-IO35-Pad31) -> /central_control_unit/CH5_DAIG_EN
- U4 pad 32: unconnected-(U4-IO36-Pad32) -> /central_control_unit/CH5_IN
- U4 pad 33: unconnected-(U4-IO37-Pad33) -> /central_control_unit/CH4_DAIG_EN
- U4 pad 34: unconnected-(U4-IO38-Pad34) -> /central_control_unit/CH4_IN
- U4 pad 35: unconnected-(U4-IO39-Pad35) -> /central_control_unit/CH3_DAIG_EN
- U4 pad 36: unconnected-(U4-IO40-Pad36) -> /central_control_unit/CH3_IN
- U4 pad 37: unconnected-(U4-IO41-Pad37) -> /central_control_unit/CH2_DAIG_EN
- U4 pad 38: unconnected-(U4-IO42-Pad38) -> /central_control_unit/CH2_IN
- U5 pad 1: /centra_control_unit/MUX_ANALOG_COM -> /central_control_unit/MUX_ANALOG_COM
- U5 pad 10: unconnected-(U5-S0-Pad10) -> /central_control_unit/MUX_S0
- U5 pad 11: unconnected-(U5-S1-Pad11) -> /central_control_unit/MUX_S1
- U5 pad 13: unconnected-(U5-S3-Pad13) -> /central_control_unit/MUX_S3
- U5 pad 14: unconnected-(U5-S2-Pad14) -> /central_control_unit/MUX_S2
- U5 pad 5: /centra_control_unit/CH5_DIAG -> /central_control_unit/CH5_DIAG
- U5 pad 6: /centra_control_unit/CH4_DIAG -> /central_control_unit/CH4_DIAG
- U9 pad 4: /centra_control_unit/CH4_DIAG -> /central_control_unit/CH4_DIAG
Routing:
- net /central_control_unit/CH1_DIAG: track 0.00 -> 48.0 mm
- net /central_control_unit/CH2_DIAG: track 0.00 -> 40.0 mm
- net /central_control_unit/CH3_DIAG: track 0.00 -> 32.4 mm
- net unconnected-(U11-WARNING-Pad8): track 0.00 -> 30.7 mm
- net unconnected-(U11-CRITICAL-Pad9): track 0.00 -> 29.2 mm
- net unconnected-(U11-PV-Pad10): track 0.00 -> 29.1 mm
- net /central_control_unit/SCL: track 0.00 -> 28.9 mm
- net /central_control_unit/SDA: track 0.00 -> 28.6 mm
- net /central_control_unit/CH4_DIAG: track 0.00 -> 24.5 mm
- net /high_power/RSH5_LO: track 0.00 -> 19.4 mm, vias 0 -> 1
- net /high_power/RSH5_HI: track 0.00 -> 18.9 mm, vias 0 -> 1
- net Net-(U6-DEN): track 0.00 -> 17.9 mm, vias 0 -> 2
- net /central_control_unit/CH5_DIAG: track 0.00 -> 16.9 mm
- net Net-(U6-IN): track 0.00 -> 16.9 mm, vias 0 -> 2
- net Net-(U7-DEN): track 0.00 -> 15.2 mm, vias 0 -> 2
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- added copper zone on B.Cu, net /central_control_unit/V_Bat
- added copper zone on F.Cu, net /central_control_unit/V_Bat
- added copper zone on F.Cu, net Net-(Battery1-Pad1)
- added copper zone on B.Cu, net Net-(F1-Pad1)
- added copper zone on F.Cu, net Net-(F1-Pad1)
- added copper zone on F.Cu, net Net-(Inverter1-Pad1)
- added copper zone on B.Cu, net Net-(J3-Pin_1)
- added copper zone on B.Cu, net Net-(J3-Pin_2)
- added copper zone on B.Cu, net Net-(J3-Pin_3)
- added copper zone on B.Cu, net Net-(J3-Pin_4)
- added copper zone on B.Cu, net Net-(J3-Pin_5)
- added copper zone on B.Cu, net Net-(J4-Pin_1)
- added copper zone on F.Cu, net Net-(J4-Pin_1)
- added copper zone on B.Cu, net Net-(J4-Pin_2)
- added copper zone on F.Cu, net Net-(J4-Pin_2)
- added copper zone on B.Cu, net Net-(J4-Pin_3)
- added copper zone on F.Cu, net Net-(J4-Pin_3)
Other:
- board size 100 x 100 mm -> 155.2 x 120 mm

Commit message: hss GPIO implemented, compiling fine
Parts:
- moved J2 53.9 mm to (98.4, 134.0)
- moved R3 53.9 mm to (96.9, 101.3)
- moved U2 53.9 mm to (97.9, 109.5)
- moved U3 53.9 mm to (97.9, 124.0)
- moved C1 53.9 mm to (101.2, 101.3)
- moved C4 53.9 mm to (96.6, 115.3)
- moved R4 53.9 mm to (92.6, 101.3)
Changed lines of the file:
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@@
 			(outputformat 1)
 			(mirror no)
-			(drillshape 1)
+			(drillshape 0)
 			(scaleselection 1)
-			(outputdirectory "")
+			(outputdirectory "outputs/")
 		)
 	)
@@
 		)
 		(fp_text user "${REFERENCE}"
-			(at 0 2.54 360)
+			(at 0 2.54 0)
 			(layer "F.Fab")
 			(effects
@@
 	(footprint "TerminalBlock:TerminalBlock_Xinya_XY308-2.54-2P_1x02_P2.54mm_Horizontal"
 		(layer "F.Cu")
-		(at 152.25 131.15)
+		(at 98.405 133.975)
 		(descr "Terminal Block Xinya XY308-2.54-2P, 2 pins, pitch 2.54mm, size 5.58x6.5mm^2, drill diameter 1.2mm, pad diameter 2mm, see http://www.xinyaelectronic.com/product/xy308-254, script-generated using https://gitlab.com/kicad/libraries/kicad-footprint-generator/-/tree/master/scripts/TerminalBlock_Xinya")
 		(tags "THT Terminal Block Xinya XY308-2.54-2P pitch 2.54mm size 5.58x6.5mm^2 drill 1.2mm pad 2mm")
@@
 		(tags "resistor handsolder")
 		(property "Reference" "R15"
-			(at 0 1.82 360)
+			(at 0 1.82 0)
 			(layer "B.SilkS")
 			(effects
@@
 		)
 		(property "Value" "4.7k"
-			(at 0 -1.82 360)
+			(at 0 -1.82 0)
 			(layer "B.Fab")
 			(effects
@@
 		)
 		(fp_text user "${REFERENCE}"
-			(at 0 0 360)
+			(at 0 0 0)
 			(layer "B.Fab")
 			(effects
@@
 		(tags "resistor handsolder")
 		(property "Reference" "R10"
-			(at -4 -0.5 360)
+			(at -4 -0.5 0)
 			(layer "B.SilkS")
 			(effects
@@
 		)
 		(property "Value" "10 ohm"
-			(at 0 -1.65 360)
+			(at 0 -1.65 0)
 			(layer "B.Fab")
 			(effects
@@
 		)
 		(fp_text user "${REFERENCE}"
-			(at 0 0 360)
+			(at 0 0 0)
 			(layer "B.Fab")
 			(effects
@@
 	(footprint "Package_SO:SOIC-8_3.9x4.9mm_P1.27mm"
 		(layer "B.Cu")
-		(at 151.75 121.15 -90)
+		(at 97.905 123.975 -90)
 		(descr "SOIC, 8 Pin (JEDEC MS-012AA, https://www.analog.com/media/en/package-pcb-resources/package/pkg_pdf/soic_narrow-r/r_8.pdf), generated with kicad-footprint-generator ipc_gullwing_generator.py")
 		(tags "SOIC SO")
@@
 	(footprint "Capacitor_SMD:C_0805_2012Metric_Pad1.18x1.45mm_HandSolder"
 		(layer "B.Cu")
-		(at 150.45 112.5)
+		(at 96.605 115.325)
 		(descr "Capacitor SMD 0805 (2012 Metric), square (rectangular) end terminal, IPC_7351 nominal with elongated pad for handsoldering. (Body size source: IPC-SM-782 page 76, https://www.pcb-3d.com/wordpress/wp-content/uploads/ipc-sm-782a_amendment_1_and_2.pdf, https://docs.google.com/spreadsheets/d/1BsfQQcO9C6DZCsRaXUlFlo91Tg2WpOkGARC1WS5S8t0/edit?usp=sharing), generated with kicad-footprint-generator")
 		(tags "capacitor handsolder")
@@
 	(footprint "Package_TO_SOT_SMD:SOT-223-3_TabPin2"
 		(layer "B.Cu")
-		(at 151.75 106.65 -90)
+		(at 97.905 109.475 -90)
 		(descr "module CMS SOT223 4 pins")
 		(tags "CMS SOT")
@@
 		(tags "SSOP 0.65")
 		(property "Reference" "U5"
-			(at 0 5.25 360)
+			(at 0 5.25 0)
 			(layer "B.SilkS")
 			(effects
@@
 		)
 		(property "Value" "CD74HC4067SM"
-			(at 0 -5.25 360)
+			(at 0 -5.25 0)
 			(layer "B.Fab")
 			(effects
@@
 		)
 		(fp_text user "${REFERENCE}"
-			(at 0 0 360)
+			(at 0 0 0)
 			(layer "B.Fab")
 			(effects
@@
 	(footprint "Resistor_SMD:R_0805_2012Metric_Pad1.20x1.40mm_HandSolder"
 		(layer "B.Cu")
-		(at 150.75 98.5 180)
+		(at 96.905 101.325 180)
 		(descr "Resistor SMD 0805 (2012 Metric), square (rectangular) end terminal, IPC_7351 nominal with elongated pad for handsoldering. (Body size source: IPC-SM-782 page 72, https://www.pcb-3d.com/wordpress/wp-content/uploads/ipc-sm-782a_amendment_1_and_2.pdf), generated with kicad-footprint-generator")
 		(tags "resistor handsolder")
@@
 		(tags "resistor handsolder")
 		(property "Reference" "R11"
-			(at -3.5 0.5 360)
+			(at -3.5 0.5 0)
 			(layer "B.SilkS")
 			(effects
@@
 		)
 		(property "Value" "10 ohm"
-			(at 0 -1.65 360)
+			(at 0 -1.65 0)
 			(layer "B.Fab")
 			(effects
@@
 		)
 		(fp_text user "${REFERENCE}"
-			(at 0 0 360)
+			(at 0 0 0)
 			(layer "B.Fab")
 			(effects
@@
 	(footprint "Capacitor_SMD:C_0805_2012Metric_Pad1.18x1.45mm_HandSolder"
 		(layer "B.Cu")
-		(at 155.0125 98.5)
+		(at 101.1675 101.325)
 		(descr "Capacitor SMD 0805 (2012 Metric), square (rectangular) end terminal, IPC_7351 nominal with elongated pad for handsoldering. (Body size source: IPC-SM-782 page 76, https://www.pcb-3d.com/wordpress/wp-content/uploads/ipc-sm-782a_amendment_1_and_2.pdf, https://docs.google.com/spreadsheets/d/1BsfQQcO9C6DZCsRaXUlFlo91Tg2WpOkGARC1WS5S8t0/edit?usp=sharing), generated with kicad-footprint-generator")
 		(tags "capacitor handsolder")
@@
 		(tags "capacitor handsolder")
 		(property "Reference" "C7"
-			(at 3 0 360)
+			(at 3 0 0)
 			(layer "B.SilkS")
 			(effects
@@
 		)
 		(property "Value" "1uF"
-			(at 0 -1.68 360)
+			(at 0 -1.68 0)
 			(layer "B.Fab")
 			(effects
@@
 		)
 		(fp_text user "${REFERENCE}"
-			(at 0 0 360)
+			(at 0 0 0)
 			(layer "B.Fab")
 			(effects
@@
 		(tags "capacitor handsolder")
 		(property "Reference" "C8"
-			(at 0 1.68 360)
+			(at 0 1.68 0)
 			(layer "B.SilkS")
 			(effects
@@
 		)
 		(property "Value" "1uF"
-			(at 0 -1.68 360)
+			(at 0 -1.68 0)
 			(layer "B.Fab")
 			(effects
@@
 		)
 		(fp_text user "${REFERENCE}"
-			(at 0 0 360)
+			(at 0 0 0)
 			(layer "B.Fab")
 			(effects
@@
 	(footprint "Resistor_SMD:R_0805_2012Metric_Pad1.20x1.40mm_HandSolder"
 		(layer "B.Cu")
-		(at 146.45 98.5 180)
+		(at 92.605 101.325 180)
 		(descr "Resistor SMD 0805 (2012 Metric), square (rectangular) end terminal, IPC_7351 nominal with elongated pad for handsoldering. (Body size source: IPC-SM-782 page 72, https://www.pcb-3d.com/wordpress/wp-content/uploads/ipc-sm-782a_amendment_1_and_2.pdf), generated with kicad-footprint-generator")
 		(tags "resistor handsolder")
@@
 		(min_thickness 0.25)
 		(filled_areas_thickness no)
-		(fill
+		(fill yes
 			(thermal_gap 0.5)
 			(thermal_bridge_width 0.5)

Commit message: lisbon flight changes
Changed lines of the file:
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@@
 		(polygon
 			(pts
-				(xy 73.5 49.254164) (xy 75.495692 49.254164) (xy 76.995692 49.254164) (xy 82.495692 49.354164) (xy 102.495692 49.354164)
-				(xy 106.495692 49.254164) (xy 106.495692 70.5) (xy 75.995692 70.5) (xy 76 60.5) (xy 74.5 58.5) (xy 74 55.254164)
+				(xy 88.754308 50.254164) (xy 90.75 50.254164) (xy 92.25 50.254164) (xy 97.75 50.354164) (xy 117.75 50.354164)
+				(xy 121.75 50.254164) (xy 121.75 71.5) (xy 91.25 71.5) (xy 91.254308 61.5) (xy 89.754308 59.5) (xy 89.254308 56.254164)
 			)
 		)
@@
 		(polygon
 			(pts
-				(xy 76 70.5) (xy 106.5 70.5) (xy 106.5 49.5) (xy 73.5 49.5) (xy 74.5 58.5) (xy 76 61)
-			)
-		)
+				(xy 89.75 71) (xy 120.25 71) (xy 120.25 50) (xy 87.25 50) (xy 88.25 59) (xy 89.75 61.5)
+			)
+		)

Commit message: flight back. different layout. start analog ui
Parts:
- removed C_GND1, C_GND2, C_GND3, C_GND4, C_GND5: 10nF, Capacitor_SMD:C_0805_2012Metric_Pad1.18x1.45mm_HandSolder
- removed J5: 12V_BusBar, HeavyDuty:half_busbar-15mm
- removed U5: CD74HC4067SM, Package_SO:SSOP-24_5.3x8.2mm_P0.65mm
- added C9: 4.7uF, Capacitor_SMD:C_0805_2012Metric_Pad1.18x1.45mm_HandSolder, F.Cu at (251.4, 116.2)
- added D10: WS2812B, LED_SMD:LED_WS2812B-Mini_PLCC4_3.5x3.5mm, F.Cu at (216.8, 139.1)
- added D11: WS2812B, LED_SMD:LED_WS2812B-Mini_PLCC4_3.5x3.5mm, F.Cu at (216.8, 145.1)
- added D16: WS2812B, LED_SMD:LED_WS2812B-Mini_PLCC4_3.5x3.5mm, F.Cu at (230.0, 98.2)
- added D17: WS2812B, LED_SMD:LED_WS2812B-Mini_PLCC4_3.5x3.5mm, F.Cu at (231.4, 143.9)
- added D18: WS2812B, LED_SMD:LED_WS2812B-Mini_PLCC4_3.5x3.5mm, F.Cu at (231.1, 118.3)
- added D19: WS2812B, LED_SMD:LED_WS2812B-Mini_PLCC4_3.5x3.5mm, F.Cu at (231.1, 124.9)
- added D2: 1N4148W, Diode_SMD:D_SOD-123, F.Cu at (244.7, 110.4)
- added D20: WS2812B, LED_SMD:LED_WS2812B-Mini_PLCC4_3.5x3.5mm, F.Cu at (231.1, 131.5)
- added D21: WS2812B, LED_SMD:LED_WS2812B-Mini_PLCC4_3.5x3.5mm, F.Cu at (231.1, 138.1)
- added D3: WS2812B, LED_SMD:LED_WS2812B-Mini_PLCC4_3.5x3.5mm, F.Cu at (216.6, 92.9)
- added D4: WS2812B, LED_SMD:LED_WS2812B-Mini_PLCC4_3.5x3.5mm, F.Cu at (216.6, 98.4)
- added D5: WS2812B, LED_SMD:LED_WS2812B-Mini_PLCC4_3.5x3.5mm, F.Cu at (216.6, 103.9)
- added D6: WS2812B, LED_SMD:LED_WS2812B-Mini_PLCC4_3.5x3.5mm, F.Cu at (216.6, 109.4)
- added D7: WS2812B, LED_SMD:LED_WS2812B-Mini_PLCC4_3.5x3.5mm, F.Cu at (230.2, 107.0)
- added D8: WS2812B, LED_SMD:LED_WS2812B-Mini_PLCC4_3.5x3.5mm, F.Cu at (216.8, 127.0)
- added D9: WS2812B, LED_SMD:LED_WS2812B-Mini_PLCC4_3.5x3.5mm, F.Cu at (216.8, 133.0)
- added F3: 20A, HeavyDuty:ATO_fuse_holder, F.Cu at (92.8, 46.1)
- added F5: 20A, HeavyDuty:ATO_fuse_holder, F.Cu at (102.0, 46.1)
- added FB2: FerriteBead 47 Ohm, Inductor_SMD:L_Walsin_WLFM201609x, B.Cu at (125.5, 85.3)
- added J10: CH2, HeavyDuty:keystone_m3_screw_terminal_vertical, F.Cu at (42.9, 116.3)
- added J12: Conn_01x01, HeavyDuty:keystone_m3_screw_terminal_vertical, F.Cu at (139.2, 25.5)
- added J13: CH3, HeavyDuty:keystone_m3_screw_terminal_vertical, F.Cu at (55.1, 116.3)
- added J14: CH4, HeavyDuty:keystone_m3_screw_terminal_vertical, F.Cu at (67.3, 116.3)
- added J15: CH5, HeavyDuty:keystone_m3_screw_terminal_vertical, F.Cu at (79.3, 116.3)
- added J16: Conn_01x02, TerminalBlock:TerminalBlock_Xinya_XY308-2.54-2P_1x02_P2.54mm_Horizontal, F.Cu at (100.3, 107.6)
- added J17: Conn_01x03, TerminalBlock:TerminalBlock_Xinya_XY308-2.54-3P_1x03_P2.54mm_Horizontal, F.Cu at (112.0, 88.2)
- added J18: Conn_01x03, TerminalBlock:TerminalBlock_Xinya_XY308-2.54-3P_1x03_P2.54mm_Horizontal, F.Cu at (112.0, 97.5)
- added J19: Conn_01x03, TerminalBlock:TerminalBlock_Xinya_XY308-2.54-3P_1x03_P2.54mm_Horizontal, F.Cu at (112.3, 107.1)
- added J20: water_sensor_conn, TerminalBlock:TerminalBlock_Xinya_XY308-2.54-5P_1x05_P2.54mm_Horizontal, F.Cu at (96.9, 117.1)
- added J21: Conn_01x02, TerminalBlock:TerminalBlock_Xinya_XY308-2.54-2P_1x02_P2.54mm_Horizontal, F.Cu at (243.2, 152.4)
- added J22: Conn_01x02, TerminalBlock:TerminalBlock_Xinya_XY308-2.54-2P_1x02_P2.54mm_Horizontal, F.Cu at (250.7, 152.5)
- added J23: Conn_01x01, HeavyDuty:keystone_m3_screw_terminal_vertical, F.Cu at (80.8, 25.2)
- added J24: Conn_01x01, HeavyDuty:keystone_m3_screw_terminal_vertical, F.Cu at (93.8, 25.2)
- added J25: Conn_01x08, TerminalBlock:TerminalBlock_Xinya_XY308-2.54-8P_1x08_P2.54mm_Horizontal, F.Cu at (205.5, 119.2)
- added J8: Conn_01x01, HeavyDuty:keystone_m3_screw_terminal_vertical, F.Cu at (126.2, 25.5)
- added Q1: Q_PMOS_GDS, Package_TO_SOT_SMD:SOT-23_Handsoldering, B.Cu at (95.8, 97.1)
- added Q2: AON6407-HXZ, Package_TO_SOT_SMD:SOT-23, F.Cu at (250.3, 82.1)
- added Q3: N-MOS, Package_TO_SOT_SMD:SOT-23, B.Cu at (124.8, 99.8)
- added Q4: N-MOS, Package_TO_SOT_SMD:SOT-23, B.Cu at (124.8, 108.3)
- added Q5: N-MOS, Package_TO_SOT_SMD:SOT-23, B.Cu at (124.8, 104.1)
- added R17: 1k, Resistor_SMD:R_0805_2012Metric_Pad1.20x1.40mm_HandSolder, B.Cu at (91.6, 95.6)
- added R18: 4.7k, Resistor_SMD:R_0805_2012Metric_Pad1.20x1.40mm_HandSolder, B.Cu at (129.8, 100.8)
- added R19: 4.7k, Resistor_SMD:R_0805_2012Metric_Pad1.20x1.40mm_HandSolder, B.Cu at (129.8, 105.0)
- added R20: 4.7k, Resistor_SMD:R_0805_2012Metric_Pad1.20x1.40mm_HandSolder, B.Cu at (129.8, 109.3)
- added R21: 4.7k, Resistor_SMD:R_0805_2012Metric_Pad1.20x1.40mm_HandSolder, B.Cu at (116.1, 81.1)
- added R22: 50 Ohm, Resistor_SMD:R_0805_2012Metric_Pad1.20x1.40mm_HandSolder, F.Cu at (250.4, 107.9)
- added R23: 100k, Resistor_THT:R_Axial_DIN0207_L6.3mm_D2.5mm_P7.62mm_Horizontal, F.Cu at (242.9, 142.5)
- added R24: 100k, Resistor_THT:R_Axial_DIN0207_L6.3mm_D2.5mm_P7.62mm_Horizontal, F.Cu at (248.2, 142.5)
- added R25: 4.7kΩ, Resistor_SMD:R_0805_2012Metric_Pad1.20x1.40mm_HandSolder, F.Cu at (250.4, 110.9)
- added R26: 4.7k, Resistor_SMD:R_0805_2012Metric_Pad1.20x1.40mm_HandSolder, B.Cu at (91.6, 93.3)
- added R28: 4.7k, Resistor_SMD:R_0805_2012Metric_Pad1.20x1.40mm_HandSolder, B.Cu at (106.8, 82.8)
- added R29: 4.7k, Resistor_SMD:R_0805_2012Metric_Pad1.20x1.40mm_HandSolder, B.Cu at (103.8, 82.8)
- added R30: 4.7k, Resistor_SMD:R_0805_2012Metric_Pad1.20x1.40mm_HandSolder, B.Cu at (100.8, 82.8)
- added R31: 4.7k, Resistor_SMD:R_0805_2012Metric_Pad1.20x1.40mm_HandSolder, B.Cu at (97.9, 82.8)
- added R32: 4.7k, Resistor_SMD:R_0805_2012Metric_Pad1.20x1.40mm_HandSolder, B.Cu at (95.0, 82.8)
- added RL1: AZSR131-1AE-12D, HeavyDuty:PRE29-same-sky, F.Cu at (257.9, 133.4)
- added SW1: SW_Push, analog_ui:button_12mm, F.Cu at (193.0, 95.0)
- added SW2: SW_Push, analog_ui:button_12mm, F.Cu at (193.0, 108.0)
- added SW3: SW_Push, analog_ui:button_12mm, F.Cu at (193.0, 121.0)
- added SW4: SW_Push, analog_ui:button_12mm, F.Cu at (193.0, 134.0)
- added SW5: SW_Push, analog_ui:button_12mm, F.Cu at (193.0, 147.0)
- added U13: CNY17-1, Package_TO_SOT_SMD:SOT-23-6, F.Cu at (244.8, 115.2)
- added U15: TCA9555PWR, Package_SO:TSSOP-24_4.4x7.8mm_P0.65mm, B.Cu at (40.9, 82.6)
- added U16: ULN2003, Package_SO:SO-16_3.9x9.9mm_P1.27mm, B.Cu at (102.1, 90.1)
- added U17: H11AA1, Package_DIP:DIP-6_W7.62mm, F.Cu at (243.2, 128.2)
- Battery1: footprint HeavyDuty:high_current_pad -> HeavyDuty:small_busbar-15mm
- J1: value GND NetTie -> rgb_led_conn; footprint Connector_PinHeader_1.00mm:PinHeader_1x02_P1.00mm_Vertical -> TerminalBlock:TerminalBlock_Xinya_XY308-2.54-3P_1x03_P2.54mm_Horizontal; moved to F.Cu
- J2: value Conn_01x02 -> CAN
- J3: value Conn 12V Out 5ch -> CH1; footprint TerminalBlock:TerminalBlock_bornier-5_P5.08mm -> HeavyDuty:keystone_m3_screw_terminal_vertical
- J4: value Chargers_Conn -> Conn_01x01; footprint HeavyDuty:3p_terminal -> HeavyDuty:keystone_m3_screw_terminal_vertical
- J6: footprint HeavyDuty:half_busbar-15mm -> HeavyDuty:small_busbar-15mm
- J9: footprint TerminalBlock:TerminalBlock_Xinya_XY308-2.54-6P_1x06_P2.54mm_Horizontal -> TerminalBlock:TerminalBlock_Xinya_XY308-2.54-5P_1x05_P2.54mm_Horizontal
- R14: value 4.7k -> 4.7k
- moved D1 155.7 mm to (254.0, 67.3), turned to -90 degrees
- moved R2 118.0 mm to (234.2, 66.2), turned to 90 degrees
- moved U1 115.4 mm to (227.9, 70.4)
- moved R1 111.8 mm to (234.2, 70.2), turned to 90 degrees
- moved C2 111.5 mm to (234.2, 74.2), turned to 90 degrees
- moved R12 50.6 mm to (109.0, 64.2), turned to -90 degrees
- moved F2 50.3 mm to (129.8, 46.1)
- moved R13 48.0 mm to (107.0, 64.2), turned to -90 degrees
- moved C5 47.7 mm to (108.0, 67.2), turned to 180 degrees
- moved R10 46.5 mm to (104.2, 64.2), turned to -90 degrees
- moved C3 45.5 mm to (87.1, 82.1), turned to -90 degrees
- moved R14 44.4 mm to (82.1, 78.3)
- moved C8 44.3 mm to (101.0, 78.8), turned to 0 degrees
- moved R15 44.3 mm to (81.8, 82.8)
- moved R11 44.1 mm to (102.2, 64.2), turned to -90 degrees
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Connections:
- net /central_control_unit/CAN_H renamed /central_control_unit/CAN/CAN_H
- net /central_control_unit/CAN_L renamed /central_control_unit/CAN/CAN_L
- C8 pad 1: GND -> GND_LP
- F1 pad 2: Net-(J4-Pin_2) -> Net-(J8-Pin_1)
- F2 pad 2: Net-(J4-Pin_3) -> Net-(J12-Pin_1)
- J1 pad 1: /central_control_unit/HP_GND -> Net-(J1-Pin_1)
- J1 pad 2: GND -> Net-(J1-Pin_2)
- J11 pad 1: Net-(J11-COM) -> /water_sensor/COM
- J11 pad 6: Net-(J11-lvl_5) -> unconnected-(J11-lvl_5-Pad6)
- J6 pad 1: GND -> GND_HP
- J7 pad 1: Net-(J7-Pin_1) -> /water_sensor/COM
- J7 pad 2: Net-(J7-Pin_2) -> unconnected-(J7-Pin_2-Pad2)
- J9 pad 1: Net-(J11-COM) -> /water_sensor/COM
- R_DEN1 pad 1: /central_control_unit/CH1_DIAG_EN -> /central_control_unit/digital_switching/CH1_DEN
- R_DEN2 pad 1: /central_control_unit/CH2_DAIG_EN -> /central_control_unit/digital_switching/CH2_DEN
- R_DEN3 pad 1: /central_control_unit/CH3_DAIG_EN -> /central_control_unit/digital_switching/CH3_DEN
- R_DEN4 pad 1: /central_control_unit/CH4_DAIG_EN -> /central_control_unit/digital_switching/CH4_DEN
- R_DEN5 pad 1: /central_control_unit/CH5_DAIG_EN -> /central_control_unit/digital_switching/CH5_DEN
- R_IN1 pad 1: /central_control_unit/CH1_IN -> /central_control_unit/digital_switching/CH1_IN
- R_IN2 pad 1: /central_control_unit/CH2_IN -> /central_control_unit/digital_switching/CH2_IN
- R_IN3 pad 1: /central_control_unit/CH3_IN -> /central_control_unit/digital_switching/CH3_IN
- R_IN4 pad 1: /central_control_unit/CH4_IN -> /central_control_unit/digital_switching/CH4_IN
- R_IN5 pad 1: /central_control_unit/CH5_IN -> /central_control_unit/digital_switching/CH5_IN
- U10 pad 1: /central_control_unit/HP_GND -> GND_HP
- U10 pad 10: Net-(J3-Pin_5) -> Net-(J15-Pin_1)
- U10 pad 12: Net-(J3-Pin_5) -> Net-(J15-Pin_1)
- U10 pad 13: Net-(J3-Pin_5) -> Net-(J15-Pin_1)
- U10 pad 14: Net-(J3-Pin_5) -> Net-(J15-Pin_1)
- U10 pad 15: /central_control_unit/V_Bat -> /central_control_unit/digital_switching/V_Bat
- U10 pad 4: /central_control_unit/CH5_DIAG -> /central_control_unit/ch5_diag
- U10 pad 8: Net-(J3-Pin_5) -> Net-(J15-Pin_1)
- U10 pad 9: Net-(J3-Pin_5) -> Net-(J15-Pin_1)
- U11 pad 3: GND -> GND_LP
- U11 pad 5: GND -> GND_LP
- U12 pad 1: Net-(J7-Pin_1) -> unconnected-(U12-COM-Pad1)
- U12 pad 2: Net-(J7-Pin_2) -> unconnected-(U12-LVL_0-Pad2)
- U3 pad 1: /central_control_unit/CAN_TX -> /central_control_unit/CAN/CAN_TX
- U3 pad 4: /central_control_unit/CAN_RX -> /central_control_unit/CAN/CAN_RX
- U3 pad 8: /central_control_unit/CAN_SLEEP -> /central_control_unit/CAN/CAN_SLEEP
- U4 pad 1: GND -> GND_LP
- U4 pad 12: /central_control_unit/CAN_TX -> unconnected-(U4-IO8-Pad12)
- U4 pad 13: /central_control_unit/CAN_RX -> unconnected-(U4-IO9-Pad13)
- U4 pad 14: /central_control_unit/CAN_SLEEP -> unconnected-(U4-IO10-Pad14)
- U4 pad 15: unconnected-(U4-IO11-Pad15) -> /central_control_unit/230VAC/RELAY_IN
- U4 pad 16: /central_control_unit/MUX_ANALOG_COM -> /central_control_unit/230VAC/AC_DETECT
- U4 pad 17: /central_control_unit/MUX_S3 -> /central_control_unit/CAN/CAN_TX
- U4 pad 18: /central_control_unit/MUX_S2 -> /central_control_unit/CAN/CAN_RX
- U4 pad 19: /central_control_unit/MUX_S1 -> /central_control_unit/CAN/CAN_SLEEP
- U4 pad 2: GND -> GND_LP
- U4 pad 20: /central_control_unit/MUX_S0 -> /central_control_unit/temp_sensors/1-WIRE
- U4 pad 26: unconnected-(U4-IO26-Pad26) -> /central_control_unit/LED_B
- U4 pad 27: /central_control_unit/CH1_DIAG_EN -> /central_control_unit/ch4_diag
- U4 pad 28: unconnected-(U4-IO33-Pad28) -> /central_control_unit/LED_G
- U4 pad 29: unconnected-(U4-IO34-Pad29) -> /central_control_unit/LED_R
- U4 pad 30: /central_control_unit/CH1_IN -> /central_control_unit/ch5_diag
- U4 pad 31: /central_control_unit/CH5_DAIG_EN -> unconnected-(U4-IO35-Pad31)
- U4 pad 32: /central_control_unit/CH5_IN -> unconnected-(U4-IO36-Pad32)
- U4 pad 33: /central_control_unit/CH4_DAIG_EN -> unconnected-(U4-IO37-Pad33)
- U4 pad 34: /central_control_unit/CH4_IN -> unconnected-(U4-IO38-Pad34)
- U4 pad 35: /central_control_unit/CH3_DAIG_EN -> Net-(U15-~{INT})
- U4 pad 36: /central_control_unit/CH3_IN -> /central_control_unit/ch1_diag
- U4 pad 37: /central_control_unit/CH2_DAIG_EN -> /central_control_unit/ch2_diag
- U4 pad 38: /central_control_unit/CH2_IN -> /central_control_unit/ch3_diag
- U4 pad 42: GND -> GND_LP
- U4 pad 43: GND -> GND_LP
- U4 pad 46: GND -> GND_LP
- U4 pad 47: GND -> GND_LP
- U4 pad 48: GND -> GND_LP
- U4 pad 49: GND -> GND_LP
- U4 pad 50: GND -> GND_LP
- U4 pad 51: GND -> GND_LP
- U4 pad 52: GND -> GND_LP
- U4 pad 53: GND -> GND_LP
- U4 pad 54: GND -> GND_LP
- U4 pad 55: GND -> GND_LP
- U4 pad 56: GND -> GND_LP
- U4 pad 57: GND -> GND_LP
- U4 pad 58: GND -> GND_LP
- U4 pad 59: GND -> GND_LP
- U4 pad 60: GND -> GND_LP
- U4 pad 61: GND -> GND_LP
- U4 pad 62: GND -> GND_LP
- U4 pad 63: GND -> GND_LP
- U4 pad 64: GND -> GND_LP
- U4 pad 65: GND -> GND_LP
- U6 pad 1: /central_control_unit/HP_GND -> GND_HP
- U6 pad 15: /central_control_unit/V_Bat -> /central_control_unit/digital_switching/V_Bat
- U6 pad 4: /central_control_unit/CH1_DIAG -> /central_control_unit/ch1_diag
- U7 pad 1: /central_control_unit/HP_GND -> GND_HP
- U7 pad 10: Net-(J3-Pin_2) -> Net-(J10-Pin_1)
- U7 pad 12: Net-(J3-Pin_2) -> Net-(J10-Pin_1)
- U7 pad 13: Net-(J3-Pin_2) -> Net-(J10-Pin_1)
- U7 pad 14: Net-(J3-Pin_2) -> Net-(J10-Pin_1)
- U7 pad 15: /central_control_unit/V_Bat -> /central_control_unit/digital_switching/V_Bat
- U7 pad 4: /central_control_unit/CH2_DIAG -> /central_control_unit/ch2_diag
- U7 pad 8: Net-(J3-Pin_2) -> Net-(J10-Pin_1)
- U7 pad 9: Net-(J3-Pin_2) -> Net-(J10-Pin_1)
- U8 pad 1: /central_control_unit/HP_GND -> GND_HP
- U8 pad 10: Net-(J3-Pin_3) -> Net-(J13-Pin_1)
- U8 pad 12: Net-(J3-Pin_3) -> Net-(J13-Pin_1)
- U8 pad 13: Net-(J3-Pin_3) -> Net-(J13-Pin_1)
- U8 pad 14: Net-(J3-Pin_3) -> Net-(J13-Pin_1)
- U8 pad 15: /central_control_unit/V_Bat -> /central_control_unit/digital_switching/V_Bat
- U8 pad 4: /central_control_unit/CH3_DIAG -> /central_control_unit/ch3_diag
- U8 pad 8: Net-(J3-Pin_3) -> Net-(J13-Pin_1)
- U8 pad 9: Net-(J3-Pin_3) -> Net-(J13-Pin_1)
- U9 pad 1: /central_control_unit/HP_GND -> GND_HP
- U9 pad 10: Net-(J3-Pin_4) -> Net-(J14-Pin_1)
- U9 pad 12: Net-(J3-Pin_4) -> Net-(J14-Pin_1)
- U9 pad 13: Net-(J3-Pin_4) -> Net-(J14-Pin_1)
- U9 pad 14: Net-(J3-Pin_4) -> Net-(J14-Pin_1)
- U9 pad 15: /central_control_unit/V_Bat -> /central_control_unit/digital_switching/V_Bat
- U9 pad 4: /central_control_unit/CH4_DIAG -> /central_control_unit/ch4_diag
- U9 pad 8: Net-(J3-Pin_4) -> Net-(J14-Pin_1)
- U9 pad 9: Net-(J3-Pin_4) -> Net-(J14-Pin_1)
Routing:
- net /central_control_unit/CH1_DIAG: track 48.0 -> 0.00 mm
- net /central_control_unit/CH2_DIAG: track 40.0 -> 0.00 mm
- net /central_control_unit/CH3_DIAG: track 32.4 -> 0.00 mm
- net unconnected-(U11-WARNING-Pad8): track 30.7 -> 0.00 mm
- net unconnected-(U11-CRITICAL-Pad9): track 29.2 -> 0.00 mm
- net unconnected-(U11-PV-Pad10): track 29.1 -> 0.00 mm
- net /central_control_unit/SDA: track 28.6 -> 0.00 mm
- net /central_control_unit/water_sensors_logic/ws_rod_1: track 0.00 -> 27.6 mm
- net /central_control_unit/water_sensors_logic/ws_rod_2: track 0.00 -> 26.5 mm
- net /central_control_unit/water_sensors_logic/ws_rod_3: track 0.00 -> 25.2 mm
- net /central_control_unit/water_sensors_logic/ws_rod_4: track 0.00 -> 25.2 mm
- net /central_control_unit/CH4_DIAG: track 24.5 -> 0.00 mm
- net /central_control_unit/water_sensors_logic/ws_rod_0: track 0.00 -> 21.8 mm
- net /high_power/RSH5_LO: track 19.4 -> 0.00 mm, vias 1 -> 0
- net /high_power/RSH5_HI: track 18.9 -> 0.00 mm, vias 1 -> 0
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- added copper zone on B.Cu, net Net-(J10-Pin_1)
- added copper zone on F.Cu, net Net-(J10-Pin_1)
- added copper zone on B.Cu, net Net-(J12-Pin_1)
- added copper zone on F.Cu, net Net-(J12-Pin_1)
- added copper zone on B.Cu, net Net-(J13-Pin_1)
- added copper zone on F.Cu, net Net-(J13-Pin_1)
- added copper zone on B.Cu, net Net-(J14-Pin_1)
- added copper zone on F.Cu, net Net-(J14-Pin_1)
- added copper zone on B.Cu, net Net-(J15-Pin_1)
- added copper zone on F.Cu, net Net-(J15-Pin_1)
- added copper zone on F.Cu, net Net-(J3-Pin_1)
- added copper zone on B.Cu, net Net-(J8-Pin_1)
- added copper zone on F.Cu, net Net-(J8-Pin_1)
- removed copper zone on F.Cu, net Net-(Battery1-Pad1)
- removed copper zone on F.Cu, net Net-(Inverter1-Pad1)
- removed copper zone on B.Cu, net Net-(J3-Pin_2)
- removed copper zone on B.Cu, net Net-(J3-Pin_3)
- removed copper zone on B.Cu, net Net-(J3-Pin_4)
- removed copper zone on B.Cu, net Net-(J3-Pin_5)
- removed copper zone on B.Cu, net Net-(J4-Pin_2)
- removed copper zone on F.Cu, net Net-(J4-Pin_2)
- removed copper zone on B.Cu, net Net-(J4-Pin_3)
- removed copper zone on F.Cu, net Net-(J4-Pin_3)
Other:
- board size 155.2 x 120 mm -> 214.5 x 134.8 mm
- board text added: "water_sensor_logic"
