File: electronics/electronics.kicad_pcb (KiCad board)
At the start: 2 copper layers, 214.5 x 134.8 mm, 128 parts, among them J1 rgb_led_conn, J10 CH2, J12 Conn_01x01, J13 CH3, J14 CH4, J15 CH5, J16 Conn_01x02, J17 Conn_01x03, J18 Conn_01x03, J19 Conn_01x03, J2 CAN, J20 water_sensor_conn, J21 Conn_01x02, J22 Conn_01x02, J23 Conn_01x01, J24 Conn_01x01, J25 Conn_01x08, J3 CH1, J4 Conn_01x01, J6 GND_Busbar, J7 Conn_01x02, J8 Conn_01x01, J9 water_sensor_conn, Q1 Q_PMOS_GDS, Q2 AON6407-HXZ, Q3 N-MOS, Q4 N-MOS, Q5 N-MOS, SW1 SW_Push, SW2 SW_Push, SW3 SW_Push, SW4 SW_Push, SW5 SW_Push, U1 AZ1117-ADJ, U10 BTS7006, U11 INA3221, U13 CNY17-1, U15 TCA9555PWR, U16 ULN2003, U17 H11AA1, U2 AZ1117-ADJ, U3 TJA1051T-3, U4 ESP32-S3-MINI-1U, U6 BTS7006, U7 BTS7006, U8 BTS7006, U9 BTS7006

Commit message: no tracks, but placement looks good
Parts:
- removed J10: CH2, HeavyDuty:keystone_m3_screw_terminal_vertical
- removed J13: CH3, HeavyDuty:keystone_m3_screw_terminal_vertical
- removed J14: CH4, HeavyDuty:keystone_m3_screw_terminal_vertical
- removed J15: CH5, HeavyDuty:keystone_m3_screw_terminal_vertical
- removed J19: Conn_01x03, TerminalBlock:TerminalBlock_Xinya_XY308-2.54-3P_1x03_P2.54mm_Horizontal
- removed J3: CH1, HeavyDuty:keystone_m3_screw_terminal_vertical
- added J5: DB12, HeavyDuty:5p_terminal_DB12, F.Cu at (45.9, 114.0)
- C9, D2, R22, R25, U13: moved to B.Cu
- moved C1 188.4 mm to (271.3, 42.6)
- moved R3 188.4 mm to (266.9, 42.6)
- moved U2 188.4 mm to (267.2, 49.1)
- moved C4 188.4 mm to (268.9, 54.8)
- moved R4 184.8 mm to (260.4, 49.0)
- moved C3 134.7 mm to (221.0, 67.0)
- moved J22 107.1 mm to (150.2, 115.3)
- moved J21 107.1 mm to (142.7, 115.2)
- moved R23 104.6 mm to (144.5, 107.3)
- moved R24 103.4 mm to (151.0, 107.3)
- moved RL1 102.6 mm to (161.5, 98.5)
- moved U17 102.5 mm to (146.0, 95.8)
- moved R22 98.3 mm to (155.5, 82.5), turned to -90 degrees
- moved C9 91.4 mm to (166.5, 82.5), turned to 90 degrees
- moved U13 91.4 mm to (159.5, 82.5)
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Connections:
- net Net-(J21-Pin_1) renamed /central_control_unit/230VAC/P_230VAC
- net Net-(J21-Pin_2) renamed /central_control_unit/230VAC/N_230VAC
- C1 pad 2: GND -> GND_LP
- C2 pad 1: GND -> GND_LP
- C9 pad 2: GND -> GND_LP
- D1 pad 2: /central_control_unit/V_Bat -> V_Bat
- F3 pad 1: /central_control_unit/V_Bat -> V_Bat
- F5 pad 1: /central_control_unit/V_Bat -> V_Bat
- J11 pad 1: /water_sensor/COM -> Net-(J11-COM)
- J7 pad 1: /water_sensor/COM -> Net-(J7-Pin_1)
- J7 pad 2: unconnected-(J7-Pin_2-Pad2) -> Net-(J7-Pin_2)
- J9 pad 1: /water_sensor/COM -> Net-(J11-COM)
- MH1 pad 1: GND -> GND_HP
- MH2 pad 1: GND -> GND_HP
- MH3 pad 1: GND -> GND_HP
- MH4 pad 1: GND -> GND_HP
- R2 pad 2: GND -> GND_LP
- R21 pad 1: +3V3 -> Net-(R21-Pad1)
- R4 pad 2: Net-(R4-Pad2) -> GND_LP
- R5 pad 4: /central_control_unit/V_Bat -> V_Bat
- R6 pad 4: /central_control_unit/V_Bat -> V_Bat
- R8 pad 4: /central_control_unit/V_Bat -> V_Bat
- U10 pad 15: /central_control_unit/digital_switching/V_Bat -> V_Bat
- U12 pad 1: unconnected-(U12-COM-Pad1) -> Net-(J7-Pin_1)
- U12 pad 2: unconnected-(U12-LVL_0-Pad2) -> Net-(J7-Pin_2)
- U15 pad 24: unconnected-(U15-VCC-Pad24) -> +3.3V
- U17 pad 4: GND -> GND_LP
- U6 pad 15: /central_control_unit/digital_switching/V_Bat -> V_Bat
- U7 pad 15: /central_control_unit/digital_switching/V_Bat -> V_Bat
- U8 pad 15: /central_control_unit/digital_switching/V_Bat -> V_Bat
- U9 pad 15: /central_control_unit/digital_switching/V_Bat -> V_Bat
Routing:
- net /central_control_unit/water_sensors_logic/ws_rod_1: track 27.6 -> 0.00 mm
- net /central_control_unit/water_sensors_logic/ws_rod_2: track 26.5 -> 0.00 mm
- net /central_control_unit/water_sensors_logic/ws_rod_3: track 25.2 -> 0.00 mm
- net /central_control_unit/water_sensors_logic/ws_rod_4: track 25.2 -> 0.00 mm
- net /central_control_unit/water_sensors_logic/ws_rod_0: track 21.8 -> 0.00 mm
- net /central_control_unit/water_sensors_logic/grey_water_rod: track 16.5 -> 0.00 mm, vias 1 -> 0
- net /central_control_unit/SCL: track 15.3 -> 0.00 mm
- net Net-(C3-Pad1): track 13.5 -> 0.00 mm
- net /central_control_unit/digital_switching/CH1_IN: track 11.7 -> 0.00 mm
- net /central_control_unit/digital_switching/CH1_DEN: track 10.2 -> 0.00 mm
- net /central_control_unit/ch1_diag: track 5.86 -> 0.00 mm
- net /central_control_unit/ch2_diag: track 4.79 -> 0.00 mm
- net Net-(U6-IN): track 4.02 -> 0.00 mm
- net Net-(U8-IN): track 3.90 -> 0.00 mm
- net Net-(U10-IN): track 3.79 -> 0.00 mm
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- added copper zone on B.Cu, net Net-(Battery1-Pad1)
- added copper zone on F.Cu, net Net-(Battery1-Pad1)
- added copper zone on B.Cu, net V_Bat
- added copper zone on F.Cu, net V_Bat
- removed copper zone on B.Cu, net /central_control_unit/V_Bat
- removed copper zone on F.Cu, net /central_control_unit/V_Bat
- removed copper zone on B.Cu, net Net-(J5-Pin_1)
- removed copper zone on F.Cu, net Net-(J5-Pin_1)
- removed copper zone on B.Cu, net Net-(J5-Pin_2)
- removed copper zone on F.Cu, net Net-(J5-Pin_2)
- removed copper zone on B.Cu, net Net-(J5-Pin_3)
- removed copper zone on F.Cu, net Net-(J5-Pin_3)
- removed copper zone on B.Cu, net Net-(J5-Pin_4)
- removed copper zone on F.Cu, net Net-(J5-Pin_4)
- removed copper zone on B.Cu, net Net-(J5-Pin_5)
- removed copper zone on F.Cu, net Net-(J5-Pin_5)
Other:
- board text added: "1-Wire"
- board text added: "Digital Switching"
- board text added: "Power Monitoring"
- board text added: "RGB_LED logic"
- board text added: "~ 230VAC"

Commit message: nerd weekend update
Parts:
- U16: moved to F.Cu

Commit message: start to create BOM and finalising symbol fields
Parts:
- removed Battery1: ~, HeavyDuty:small_busbar-15mm
- removed FB2: FerriteBead 47 Ohm, Inductor_SMD:L_Walsin_WLFM201609x
- removed Inverter1: ~, HeavyDuty:high_current_pad
- removed Q5: N-MOS, Package_TO_SOT_SMD:SOT-23
- removed U2: AZ1117-ADJ, Package_TO_SOT_SMD:SOT-223-3_TabPin2
- added C10: 22uF, Capacitor_SMD:C_0805_2012Metric, B.Cu at (67.5, 79.5)
- added C10: 22uF, Capacitor_SMD:C_0805_2012Metric_Pad1.18x1.45mm_HandSolder, B.Cu at (89.0, 78.0)
- added C11: 100nF, Capacitor_SMD:C_0805_2012Metric, B.Cu at (84.5, 101.0)
- added C12: 100nF, Capacitor_SMD:C_0805_2012Metric, B.Cu at (89.5, 109.0)
- added C13: C_Polarized, Capacitor_THT:CP_Radial_D5.0mm_P2.50mm, F.Cu at (174.0, 99.2)
- added C14: C, Capacitor_SMD:C_0805_2012Metric, B.Cu at (172.7, 111.2)
- added C15: 1uF, Capacitor_SMD:C_0805_2012Metric, B.Cu at (95.5, 93.0)
- added C16: C_Polarized, Capacitor_THT:CP_Radial_D5.0mm_P2.50mm, F.Cu at (100.0, 105.0)
- added C17: 10uF, Capacitor_SMD:C_0805_2012Metric, F.Cu at (54.5, 223.0)
- added C18: 10uF, Capacitor_SMD:C_0805_2012Metric, F.Cu at (54.5, 226.0)
- added C19: 10uF, Capacitor_SMD:C_0805_2012Metric, F.Cu at (54.5, 229.0)
- added C20: 10uF, Capacitor_SMD:C_0805_2012Metric, F.Cu at (54.5, 232.0)
- added C21: 10uF, Capacitor_SMD:C_0805_2012Metric, F.Cu at (54.5, 235.0)
- added C22: C_Polarized, Capacitor_THT:CP_Radial_D5.0mm_P2.50mm, F.Cu at (81.9, 221.4)
- added C23: C_Polarized, Capacitor_THT:CP_Radial_D5.0mm_P2.50mm, F.Cu at (81.4, 227.9)
- added C24: C_Polarized, Capacitor_THT:CP_Radial_D5.0mm_P2.50mm, F.Cu at (81.9, 235.9)
- added C25: 10uF, Capacitor_SMD:C_0805_2012Metric, B.Cu at (89.5, 104.0)
- added C26: C_Polarized, Capacitor_THT:CP_Radial_D5.0mm_P2.50mm, F.Cu at (93.8, 105.0)
- added C27: 100nF, Capacitor_SMD:C_0805_2012Metric, B.Cu at (89.5, 106.5)
- added C28: C_Polarized, Capacitor_THT:CP_Radial_D5.0mm_P2.50mm, F.Cu at (43.5, 98.2)
- added C29: C_Polarized, Capacitor_THT:CP_Radial_D5.0mm_P2.50mm, F.Cu at (67.5, 98.5)
- added C30: C_Polarized, Capacitor_THT:CP_Radial_D5.0mm_P2.50mm, F.Cu at (51.0, 98.2)
- added C31: C_Polarized, Capacitor_THT:CP_Radial_D5.0mm_P2.50mm, F.Cu at (36.5, 98.2)
- added C32: C_Polarized, Capacitor_THT:CP_Radial_D5.0mm_P2.50mm, F.Cu at (59.0, 98.5)
- added C33: C_Polarized, Capacitor_THT:CP_Radial_D5.0mm_P2.50mm, F.Cu at (114.0, 109.5)
- added D12: D_Schottky_AKA, Package_TO_SOT_SMD:TO-252-2, B.Cu at (125.5, 76.9)
- added D13: LED, LED_SMD:LED_1206_3216Metric, F.Cu at (199.5, 46.0)
- added D14: LED, LED_SMD:LED_1206_3216Metric, F.Cu at (199.5, 40.8)
- added D15: D_Schottky, Diode_SMD:D_SMA, B.Cu at (75.5, 104.0)
- added D22: D_Schottky, Diode_THT:D_DO-15_P3.81mm_Vertical_AnodeUp, F.Cu at (131.8, 76.7)
- added F6: 5A, HeavyDuty:ATO_fuse_holder, F.Cu at (132.0, 46.1)
- added FB1: FerriteBead 47 Ohm, Inductor_SMD:L_Walsin_WLFM201609x, F.Cu at (185.0, 75.5)
- added GND_Conn1: ~, HeavyDuty:small_busbar-15mm, F.Cu at (205.0, 70.0)
- added J10: water_sensor_conn, TerminalBlock:TerminalBlock_Xinya_XY308-2.54-5P_1x05_P2.54mm_Horizontal, F.Cu at (143.5, 116.0)
- added J13: Conn_01x02, TerminalBlock:TerminalBlock_Xinya_XY308-2.54-2P_1x02_P2.54mm_Horizontal, F.Cu at (143.5, 106.8)
- added J14: Conn_GND, HeavyDuty:keystone_m3_screw_terminal_vertical, F.Cu at (146.3, 25.0)
- added J15: Battery_Conn, HeavyDuty:keystone_m3_screw_terminal_vertical, F.Cu at (49.8, 25.0)
- added J26: leds_ch3, TerminalBlock:TerminalBlock_Xinya_XY308-2.54-3P_1x03_P2.54mm_Horizontal, F.Cu at (170.5, 106.8)
- added J27: leds_ch4, TerminalBlock:TerminalBlock_Xinya_XY308-2.54-3P_1x03_P2.54mm_Horizontal, F.Cu at (170.5, 116.0)
- added J28: Conn_01x08, TerminalBlock:TerminalBlock_Xinya_XY308-2.54-8P_1x08_P2.54mm_Horizontal, F.Cu at (60.1, 220.4)
- added J29: Conn_GND, HeavyDuty:keystone_m3_screw_terminal_vertical, F.Cu at (187.7, 25.0)
- added J3: Conn_01x08, TerminalBlock:TerminalBlock_Xinya_XY308-2.54-8P_1x08_P2.54mm_Horizontal, F.Cu at (91.3, 116.0)
- added J30: Conn_GND, HeavyDuty:keystone_m3_screw_terminal_vertical, F.Cu at (173.9, 25.0)
- added J31: Conn_GND, HeavyDuty:keystone_m3_screw_terminal_vertical, F.Cu at (160.1, 25.0)
- added NT1: NetTie_2, NetTie:NetTie-2_THT_Pad1.0mm, F.Cu at (130.9, 81.8)
- added R16: 100k, Resistor_SMD:R_0805_2012Metric, B.Cu at (150.6, 97.5)
- added R27: 10k, Resistor_SMD:R_0805_2012Metric, B.Cu at (95.5, 90.5)
- added R33: 4k7, Resistor_SMD:R_0805_2012Metric, B.Cu at (186.1, 35.5)
- added R34: 4k7, Resistor_SMD:R_0805_2012Metric, B.Cu at (190.1, 35.5)
- added R35: 4k7, Resistor_SMD:R_0805_2012Metric, B.Cu at (194.1, 35.5)
- added R36: 100R, Resistor_SMD:R_0805_2012Metric, B.Cu at (126.2, 84.0)
- added R37: 10k, Resistor_SMD:R_0805_2012Metric, B.Cu at (118.7, 82.0)
- added R38: 10k, Resistor_SMD:R_0805_2012Metric, B.Cu at (114.6, 81.5)
- added R39: 10k, Resistor_SMD:R_0805_2012Metric, B.Cu at (170.5, 34.0)
- added SW6: SW_DIP_x01, Connector_PinHeader_1.00mm:PinHeader_1x02_P1.00mm_Vertical, F.Cu at (79.0, 116.5)
- added SW7: RST_BTN, Button_Switch_THT:SW_PUSH_6mm_H4.3mm, F.Cu at (132.0, 104.7)
- added SW8: FLASH_BTN, Button_Switch_THT:SW_PUSH_6mm_H4.3mm, F.Cu at (132.0, 113.5)
- added U14: LM339_4ch, Package_SO:SOIC-14_3.9x8.7mm_P1.27mm, B.Cu at (144.2, 95.4)
- added U18: ~, HeavyDuty:mini360, F.Cu at (115.0, 89.0)
- added U19: ESP32-S3-MINI-1, PCM_Espressif:ESP32-S3-MINI-1U, B.Cu at (78.8, 87.7)
- added U5: LM339_4ch, Package_SO:SOIC-14_3.9x8.7mm_P1.27mm, B.Cu at (144.2, 80.8)
- C1: value 10uF -> C_Polarized; footprint Capacitor_SMD:C_0805_2012Metric_Pad1.18x1.45mm_HandSolder -> Capacitor_THT:CP_Radial_D5.0mm_P2.50mm; moved to F.Cu
- C2: value 10uF -> C; footprint Capacitor_SMD:C_0805_2012Metric_Pad1.18x1.45mm_HandSolder -> Capacitor_SMD:C_0805_2012Metric
- C3: value 22uF -> C_Polarized; footprint Capacitor_SMD:C_0805_2012Metric_Pad1.18x1.45mm_HandSolder -> Capacitor_THT:CP_Radial_D5.0mm_P2.50mm; moved to F.Cu
- C4: value 22uF -> C; footprint Capacitor_SMD:C_0805_2012Metric_Pad1.18x1.45mm_HandSolder -> Capacitor_SMD:C_0805_2012Metric
- C5, C6, C7, C8, C9: footprint Capacitor_SMD:C_0805_2012Metric_Pad1.18x1.45mm_HandSolder -> Capacitor_SMD:C_0805_2012Metric
- D1: value D -> LED; footprint Diode_SMD:D_1210_3225Metric_Pad1.42x2.65mm_HandSolder -> LED_SMD:LED_1206_3216Metric; moved to F.Cu
- D10, D11, D16, D17, D18, D19, D20, D21, D3, D4, D5, D6, D7, D8, D9: footprint LED_SMD:LED_WS2812B-Mini_PLCC4_3.5x3.5mm -> LED_SMD:LED_WS2812B_PLCC4_5.0x5.0mm_P3.2mm
- J1: value rgb_led_conn -> leds_ch1
- J16: value Conn_01x02 -> USB_C_Receptacle_USB2.0_16P; footprint TerminalBlock:TerminalBlock_Xinya_XY308-2.54-2P_1x02_P2.54mm_Horizontal -> Connector_USB:USB_C_Receptacle_JAE_DX07S016JA1R1500; moved to B.Cu
- J20: value water_sensor_conn -> leds_ch2; footprint TerminalBlock:TerminalBlock_Xinya_XY308-2.54-5P_1x05_P2.54mm_Horizontal -> TerminalBlock:TerminalBlock_Xinya_XY308-2.54-3P_1x03_P2.54mm_Horizontal
- J25: value Conn_01x08 -> Conn_GND; footprint TerminalBlock:TerminalBlock_Xinya_XY308-2.54-8P_1x08_P2.54mm_Horizontal -> HeavyDuty:keystone_m3_screw_terminal_vertical
- J6: value GND_Busbar -> Inverter_Conn; footprint HeavyDuty:small_busbar-15mm -> HeavyDuty:keystone_m3_screw_terminal_vertical
- J7: value Conn_01x02 -> grey_water_conn
- Q1: value Q_PMOS_GDS -> Q_NMOS_DGS; footprint Package_TO_SOT_SMD:SOT-23_Handsoldering -> Package_TO_SOT_SMD:SOT-323_SC-70
- Q2: value AON6407-HXZ -> Q_PMOS_DGS; footprint Package_TO_SOT_SMD:SOT-23 -> Package_TO_SOT_SMD:SOT-323_SC-70; moved to B.Cu
- Q3: value N-MOS -> Q_PMOS_DGS; footprint Package_TO_SOT_SMD:SOT-23 -> Package_TO_SOT_SMD:SOT-323_SC-70
- Q4: value N-MOS -> Q_NMOS_GDS; footprint Package_TO_SOT_SMD:SOT-23 -> Package_TO_SOT_SMD:TO-252-2
- R1: value 125 -> 10k; footprint Resistor_SMD:R_0805_2012Metric_Pad1.20x1.40mm_HandSolder -> Resistor_SMD:R_0805_2012Metric
- R10, R11, R12, R13, R21, R22, R25, R7, R9, R_DEN1, R_DEN2, R_DEN3, R_DEN4, R_DEN5, R_IN1, R_IN2, R_IN3, R_IN4, R_IN5: footprint Resistor_SMD:R_0805_2012Metric_Pad1.20x1.40mm_HandSolder -> Resistor_SMD:R_0805_2012Metric
- R14, R15: footprint Resistor_SMD:R_1206_3216Metric_Pad1.30x1.75mm_HandSolder -> Resistor_SMD:R_0805_2012Metric
- R17: value 1k -> 120; footprint Resistor_SMD:R_0805_2012Metric_Pad1.20x1.40mm_HandSolder -> Resistor_SMD:R_0805_2012Metric
- R18, R19, R20: value 4.7k -> 4k7; footprint Resistor_SMD:R_0805_2012Metric_Pad1.20x1.40mm_HandSolder -> Resistor_SMD:R_0805_2012Metric
- R2: value 205 -> 100R; footprint Resistor_SMD:R_0805_2012Metric_Pad1.20x1.40mm_HandSolder -> Resistor_SMD:R_0805_2012Metric
- R26: value 4.7k -> 100k; footprint Resistor_SMD:R_0805_2012Metric_Pad1.20x1.40mm_HandSolder -> Resistor_SMD:R_0805_2012Metric
- R28, R29, R30, R31: value 4.7k -> 1M; footprint Resistor_SMD:R_0805_2012Metric_Pad1.20x1.40mm_HandSolder -> Resistor_SMD:R_0805_2012Metric
- R3: value 125 -> 4k7; footprint Resistor_SMD:R_0805_2012Metric_Pad1.20x1.40mm_HandSolder -> Resistor_SMD:R_0805_2012Metric
- R32: value 4.7k -> 10k; footprint Resistor_SMD:R_0805_2012Metric_Pad1.20x1.40mm_HandSolder -> Resistor_SMD:R_0805_2012Metric
- R4: value 370 -> 4k7; footprint Resistor_SMD:R_0805_2012Metric_Pad1.20x1.40mm_HandSolder -> Resistor_SMD:R_0805_2012Metric
- U1: value AZ1117-ADJ -> TLV1117-33
- U10, U6, U7, U8, U9: moved to F.Cu
- U16: value ULN2003 -> ~; footprint Package_SO:SO-16_3.9x9.9mm_P1.27mm -> HeavyDuty:generic_dcdc
- U4: value ESP32-S3-MINI-1U -> ~; footprint RF_Module:ESP32-S2-MINI-1U -> HeavyDuty:generic_dcdc; moved to F.Cu
- moved SW1 231.6 mm to (25.9, 255.4), turned to 90 degrees
- moved D17 229.6 mm to (25.6, 245.7)
- moved D3 229.0 mm to (27.1, 221.4)
- moved D4 229.0 mm to (27.1, 226.9)
- moved D5 229.0 mm to (27.1, 232.4)
- moved D6 229.0 mm to (27.1, 237.9)
- moved D21 220.8 mm to (38.4, 245.9)
- moved SW2 213.3 mm to (38.9, 255.4), turned to 90 degrees
- moved D20 212.0 mm to (51.9, 244.7), turned to -90 degrees
- moved D7 207.7 mm to (65.4, 233.4), turned to -90 degrees
- moved D16 206.1 mm to (74.1, 233.2), turned to -90 degrees
- moved D19 205.2 mm to (64.5, 244.5), turned to -90 degrees
- moved D18 198.8 mm to (77.1, 243.9), turned to -90 degrees
- moved SW3 194.9 mm to (51.9, 255.4), turned to 90 degrees
- moved D8 194.0 mm to (46.3, 219.7)
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Connections:
- net Net-(J5-Pin_3) renamed /central_control_unit/digital_switching/CH3_OUT
- C1 pad 1: /central_control_unit/12V_MCU -> Net-(Q3-S)
- C1 pad 2: GND_LP -> GND_HP
- C2 pad 1: GND_LP -> Net-(Q3-S)
- C2 pad 2: /central_control_unit/12V_MCU -> GND_HP
- C3 pad 1: Net-(C3-Pad1) -> /central_control_unit/lightning/LEDS_CH12_5V
- C3 pad 2: +3.3V -> /central_control_unit/lightning/leds12_gnd
- C4 pad 1: GND -> /central_control_unit/lightning/LEDS_CH12_5V
- C4 pad 2: +5V -> /central_control_unit/lightning/leds12_gnd
- C9 pad 1: /central_control_unit/230VAC/AC_DETECT -> /central_control_unit/ac_detect
- D1 pad 1: /central_control_unit/12V_MCU -> GND_LP
- D1 pad 2: V_Bat -> Net-(D1-A)
- D10 pad 1: unconnected-(D10-VDD-Pad1) -> /analog_ui/+5V_UI
- D10 pad 2: unconnected-(D10-DOUT-Pad2) -> Net-(D10-DOUT)
- D10 pad 3: unconnected-(D10-VSS-Pad3) -> /analog_ui/GND_UI
- D10 pad 4: unconnected-(D10-DIN-Pad4) -> Net-(D10-DIN)
- D11 pad 1: unconnected-(D11-VDD-Pad1) -> /analog_ui/+5V_UI
- D11 pad 2: unconnected-(D11-DOUT-Pad2) -> Net-(D11-DOUT)
- D11 pad 3: unconnected-(D11-VSS-Pad3) -> /analog_ui/GND_UI
- D11 pad 4: unconnected-(D11-DIN-Pad4) -> Net-(D10-DOUT)
- D16 pad 1: unconnected-(D16-VDD-Pad1) -> /analog_ui/+5V_UI
- D16 pad 2: unconnected-(D16-DOUT-Pad2) -> Net-(D16-DOUT)
- D16 pad 3: unconnected-(D16-VSS-Pad3) -> /analog_ui/GND_UI
- D16 pad 4: unconnected-(D16-DIN-Pad4) -> Net-(D16-DIN)
- D17 pad 1: unconnected-(D17-VDD-Pad1) -> /analog_ui/+5V_UI
- D17 pad 2: unconnected-(D17-DOUT-Pad2) -> Net-(D17-DOUT)
- D17 pad 3: unconnected-(D17-VSS-Pad3) -> /analog_ui/GND_UI
- D17 pad 4: unconnected-(D17-DIN-Pad4) -> Net-(D16-DOUT)
- D18 pad 1: unconnected-(D18-VDD-Pad1) -> /analog_ui/+5V_UI
- D18 pad 2: unconnected-(D18-DOUT-Pad2) -> Net-(D18-DOUT)
- D18 pad 3: unconnected-(D18-VSS-Pad3) -> /analog_ui/GND_UI
- D18 pad 4: unconnected-(D18-DIN-Pad4) -> Net-(D17-DOUT)
- D19 pad 1: unconnected-(D19-VDD-Pad1) -> /analog_ui/+5V_UI
- D19 pad 2: unconnected-(D19-DOUT-Pad2) -> Net-(D19-DOUT)
- D19 pad 3: unconnected-(D19-VSS-Pad3) -> /analog_ui/GND_UI
- D19 pad 4: unconnected-(D19-DIN-Pad4) -> Net-(D18-DOUT)
- D20 pad 1: unconnected-(D20-VDD-Pad1) -> /analog_ui/+5V_UI
- D20 pad 2: unconnected-(D20-DOUT-Pad2) -> Net-(D20-DOUT)
- D20 pad 3: unconnected-(D20-VSS-Pad3) -> /analog_ui/GND_UI
- D20 pad 4: unconnected-(D20-DIN-Pad4) -> Net-(D19-DOUT)
- D21 pad 1: unconnected-(D21-VDD-Pad1) -> /analog_ui/+5V_UI
- D21 pad 3: unconnected-(D21-VSS-Pad3) -> /analog_ui/GND_UI
- D21 pad 4: unconnected-(D21-DIN-Pad4) -> Net-(D20-DOUT)
- D3 pad 1: unconnected-(D3-VDD-Pad1) -> /analog_ui/+5V_UI
- D3 pad 2: unconnected-(D3-DOUT-Pad2) -> Net-(D3-DOUT)
- D3 pad 3: unconnected-(D3-VSS-Pad3) -> /analog_ui/GND_UI
- D3 pad 4: unconnected-(D3-DIN-Pad4) -> /analog_ui/LED_DATA_IN
- D4 pad 1: unconnected-(D4-VDD-Pad1) -> /analog_ui/+5V_UI
- D4 pad 2: unconnected-(D4-DOUT-Pad2) -> Net-(D4-DOUT)
- D4 pad 3: unconnected-(D4-VSS-Pad3) -> /analog_ui/GND_UI
- D4 pad 4: unconnected-(D4-DIN-Pad4) -> Net-(D3-DOUT)
- D5 pad 1: unconnected-(D5-VDD-Pad1) -> /analog_ui/+5V_UI
- D5 pad 2: unconnected-(D5-DOUT-Pad2) -> Net-(D5-DOUT)
- D5 pad 3: unconnected-(D5-VSS-Pad3) -> /analog_ui/GND_UI
- D5 pad 4: unconnected-(D5-DIN-Pad4) -> Net-(D4-DOUT)
- D6 pad 1: unconnected-(D6-VDD-Pad1) -> /analog_ui/+5V_UI
- D6 pad 2: unconnected-(D6-DOUT-Pad2) -> Net-(D6-DOUT)
- D6 pad 3: unconnected-(D6-VSS-Pad3) -> /analog_ui/GND_UI
- D6 pad 4: unconnected-(D6-DIN-Pad4) -> Net-(D5-DOUT)
- D7 pad 1: unconnected-(D7-VDD-Pad1) -> /analog_ui/+5V_UI
- D7 pad 2: unconnected-(D7-DOUT-Pad2) -> Net-(D16-DIN)
- D7 pad 3: unconnected-(D7-VSS-Pad3) -> /analog_ui/GND_UI
- D7 pad 4: unconnected-(D7-DIN-Pad4) -> Net-(D11-DOUT)
- D8 pad 1: unconnected-(D8-VDD-Pad1) -> /analog_ui/+5V_UI
- D8 pad 3: unconnected-(D8-VSS-Pad3) -> /analog_ui/GND_UI
- D8 pad 4: unconnected-(D8-DIN-Pad4) -> Net-(D6-DOUT)
- D9 pad 1: unconnected-(D9-VDD-Pad1) -> /analog_ui/+5V_UI
- D9 pad 2: unconnected-(D9-DOUT-Pad2) -> Net-(D10-DIN)
- D9 pad 3: unconnected-(D9-VSS-Pad3) -> /analog_ui/GND_UI
- F3 pad 1: V_Bat -> +12V_HP
- F5 pad 1: V_Bat -> +12V_HP
- J1 pad 1: Net-(J1-Pin_1) -> /central_control_unit/lightning/leds12_gnd
- J1 pad 2: Net-(J1-Pin_2) -> /central_control_unit/LED_CH1
- J1 pad 3: Net-(J1-Pin_3) -> /central_control_unit/lightning/LEDS_CH12_5V
- J17 pad 2: /central_control_unit/temp_sensors/1-WIRE -> /central_control_unit/1-Wire
- J17 pad 3: GND -> GND_LP
- J18 pad 2: /central_control_unit/temp_sensors/1-WIRE -> /central_control_unit/1-Wire
- J18 pad 3: GND -> GND_LP
- J2 pad 2: /central_control_unit/CAN/CAN_L -> /central_control_unit/can_term_r_dip_2
- J20 pad 1: /central_control_unit/water_sensors_logic/ws_rod_0 -> /central_control_unit/lightning/leds12_gnd
- J20 pad 2: /central_control_unit/water_sensors_logic/ws_rod_1 -> /central_control_unit/LED_CH2
- J20 pad 3: /central_control_unit/water_sensors_logic/ws_rod_2 -> /central_control_unit/lightning/LEDS_CH12_5V
- J25 pad 1: unconnected-(J25-Pin_1-Pad1) -> GND_HP
- J5 pad 1: Net-(J5-Pin_1) -> /central_control_unit/digital_switching/CH5_OUT
- J5 pad 2: Net-(J5-Pin_2) -> /central_control_unit/digital_switching/CH4_OUT
- J5 pad 4: Net-(J5-Pin_4) -> /central_control_unit/digital_switching/CH2_OUT
- J5 pad 5: Net-(J5-Pin_5) -> /central_control_unit/digital_switching/CH1_OUT
- J6 pad 1: GND_HP -> Net-(J6-Pin_1)
- Q1 pad 1: Net-(Q1-G) -> Net-(Q1-D)
- Q1 pad 2: +3.3V -> Net-(Q1-G)
- Q1 pad 3: /central_control_unit/water_sensors_logic/ws_rod_0 -> GND_LP
- Q2 pad 1: unconnected-(Q2-G-Pad1) -> /central_control_unit/dc_dc_conversion/vin
- Q2 pad 2: unconnected-(Q2-S-Pad2) -> Net-(Q1-D)
- Q2 pad 3: unconnected-(Q2-D-Pad3) -> +12V
- Q3 pad 1: /central_control_unit/LED_R -> Net-(Q3-D)
- Q3 pad 2: Net-(J1-Pin_1) -> Net-(Q3-G)
- Q3 pad 3: GND_HP -> Net-(Q3-S)
- Q4 pad 1: /central_control_unit/LED_B -> Net-(Q3-D)
- Q4 pad 2: Net-(J1-Pin_3) -> Net-(Q4-D)
- R1 pad 1: +3.3V -> Net-(Q3-D)
- R1 pad 2: Net-(U1-ADJ) -> GND_HP
- R17 pad 1: /central_control_unit/water_sensors_logic/WS_ENABLE -> /central_control_unit/CAN/CAN_H
- R17 pad 2: Net-(Q1-G) -> /central_control_unit/can_term_r_dip_1
- R18 pad 1: /central_control_unit/LED_R -> Net-(R18-Pad1)
- R18 pad 2: GND_HP -> +5V
- R19 pad 1: /central_control_unit/LED_G -> Net-(J16-CC1)
- R19 pad 2: GND_HP -> GND_LP
- R2 pad 1: Net-(U1-ADJ) -> /central_control_unit/led_en
- R2 pad 2: GND_LP -> Net-(Q3-G)
- R20 pad 1: /central_control_unit/LED_B -> Net-(J16-CC2)
- R20 pad 2: GND_HP -> GND_LP
- R21 pad 2: /central_control_unit/temp_sensors/1-WIRE -> /central_control_unit/1-Wire
- R22 pad 1: /central_control_unit/230VAC/RELAY_IN -> /central_control_unit/relay_out
- R25 pad 2: /central_control_unit/230VAC/AC_DETECT -> /central_control_unit/ac_detect
- R26 pad 1: +3.3V -> GND_LP
- R26 pad 2: /central_control_unit/water_sensors_logic/WS_ENABLE -> /central_control_unit/water_sensors_logic/ws_vref
- R28 pad 1: +3.3V -> +3V3
- R28 pad 2: /central_control_unit/water_sensors_logic/GREY_WATER_FULL -> /central_control_unit/water_sensors_logic/probe_1
- R29 pad 1: +3.3V -> +3V3
- R29 pad 2: /central_control_unit/water_sensors_logic/WS_LVL_100% -> /central_control_unit/water_sensors_logic/probe_2
- R3 pad 1: +5V -> Net-(D14-A)
- R3 pad 2: Net-(U2-ADJ) -> Net-(R18-Pad1)
- R30 pad 1: +3.3V -> +3V3
- R30 pad 2: /central_control_unit/water_sensors_logic/WS_LVL_75% -> /central_control_unit/water_sensors_logic/probe_3
- R31 pad 1: +3.3V -> +3V3
- R31 pad 2: /central_control_unit/water_sensors_logic/WS_LVL_50% -> /central_control_unit/water_sensors_logic/probe_4
- R32 pad 2: /central_control_unit/water_sensors_logic/WS_LVL_25% -> /central_control_unit/IO_0
- R4 pad 1: Net-(U2-ADJ) -> Net-(D13-A)
- R4 pad 2: GND_LP -> +3.3V
- R5 pad 4: V_Bat -> +12V_HP
- R6 pad 4: V_Bat -> +12V_HP
- R8 pad 1: Net-(Inverter1-Pad1) -> Net-(J6-Pin_1)
- R8 pad 4: V_Bat -> +12V_HP
- R_DEN1 pad 1: /central_control_unit/digital_switching/CH1_DEN -> /central_control_unit/ch1_den
- R_DEN2 pad 1: /central_control_unit/digital_switching/CH2_DEN -> /central_control_unit/ch2_den
- R_DEN3 pad 1: /central_control_unit/digital_switching/CH3_DEN -> /central_control_unit/ch3_den
- R_DEN4 pad 1: /central_control_unit/digital_switching/CH4_DEN -> /central_control_unit/ch4_den
- R_DEN5 pad 1: /central_control_unit/digital_switching/CH5_DEN -> /central_control_unit/ch5_den
- R_IN1 pad 1: /central_control_unit/digital_switching/CH1_IN -> /central_control_unit/ch1_in
- R_IN2 pad 1: /central_control_unit/digital_switching/CH2_IN -> /central_control_unit/ch2_in
- R_IN3 pad 1: /central_control_unit/digital_switching/CH3_IN -> /central_control_unit/ch3_in
- R_IN4 pad 1: /central_control_unit/digital_switching/CH4_IN -> /central_control_unit/ch4_in
- R_IN5 pad 1: /central_control_unit/digital_switching/CH5_IN -> /central_control_unit/ch5_in
- SW1 pad 1: GND_LP -> /analog_ui/GND_UI
- SW1 pad 2: unconnected-(SW1-Pad2) -> /analog_ui/BTN_1_IN
- SW2 pad 1: GND_LP -> /analog_ui/GND_UI
- SW2 pad 2: unconnected-(SW2-Pad2) -> /analog_ui/BTN_2_IN
- SW3 pad 1: GND_LP -> /analog_ui/GND_UI
- SW3 pad 2: unconnected-(SW3-Pad2) -> /analog_ui/BTN_3_IN
- SW4 pad 1: GND_LP -> /analog_ui/GND_UI
- SW4 pad 2: unconnected-(SW4-Pad2) -> /analog_ui/BTN_4_IN
- SW5 pad 1: GND_LP -> /analog_ui/GND_UI
- SW5 pad 2: unconnected-(SW5-Pad2) -> /analog_ui/BTN_5_IN
- U1 pad 1: Net-(U1-ADJ) -> GND_LP
- U1 pad 3: /central_control_unit/12V_MCU -> +5V
- U10 pad 10: Net-(J5-Pin_5) -> /central_control_unit/digital_switching/CH5_OUT
- U10 pad 12: Net-(J5-Pin_5) -> /central_control_unit/digital_switching/CH5_OUT
- U10 pad 13: Net-(J5-Pin_5) -> /central_control_unit/digital_switching/CH5_OUT
- U10 pad 14: Net-(J5-Pin_5) -> /central_control_unit/digital_switching/CH5_OUT
- U10 pad 15: V_Bat -> +12V_HP
- U10 pad 8: Net-(J5-Pin_5) -> /central_control_unit/digital_switching/CH5_OUT
- U10 pad 9: Net-(J5-Pin_5) -> /central_control_unit/digital_switching/CH5_OUT
- U15 pad 1: Net-(U15-~{INT}) -> unconnected-(U15-~{INT}-Pad1)
- U15 pad 10: /central_control_unit/digital_switching/CH1_IN -> /central_control_unit/WS_LVL_25
- U15 pad 11: /central_control_unit/digital_switching/CH1_DEN -> /central_control_unit/can_sleep
- U15 pad 13: /central_control_unit/digital_switching/CH2_IN -> /central_control_unit/can_term_r_dip_1
- U15 pad 14: /central_control_unit/digital_switching/CH2_DEN -> /central_control_unit/can_term_r_dip_2
- U15 pad 15: /central_control_unit/digital_switching/CH3_IN -> /central_control_unit/led_en
- U15 pad 16: /central_control_unit/digital_switching/CH3_DEN -> unconnected-(U15-P13-Pad16)
- U15 pad 17: /central_control_unit/digital_switching/CH4_IN -> unconnected-(U15-P14-Pad17)
- U15 pad 18: /central_control_unit/digital_switching/CH4_DEN -> unconnected-(U15-P15-Pad18)
- U15 pad 19: /central_control_unit/digital_switching/CH5_IN -> unconnected-(U15-P16-Pad19)
- U15 pad 20: /central_control_unit/digital_switching/CH5_DEN -> unconnected-(U15-P17-Pad20)
- U15 pad 4: /central_control_unit/water_sensors_logic/WS_ENABLE -> /central_control_unit/relay_out
- U15 pad 5: /central_control_unit/water_sensors_logic/WS_LVL_25% -> /central_control_unit/ac_detect
- U15 pad 6: /central_control_unit/water_sensors_logic/WS_LVL_50% -> /central_control_unit/GREY_FULL
- U15 pad 7: /central_control_unit/water_sensors_logic/WS_LVL_75% -> /central_control_unit/WS_LVL_100
- U15 pad 8: /central_control_unit/water_sensors_logic/WS_LVL_100% -> /central_control_unit/WS_LVL_75
- U15 pad 9: /central_control_unit/water_sensors_logic/GREY_WATER_FULL -> /central_control_unit/WS_LVL_50
- U16 pad 1: /central_control_unit/water_sensors_logic/grey_water_rod -> Net-(Q3-S)
- U16 pad 2: /central_control_unit/water_sensors_logic/ws_rod_4 -> Net-(Q4-D)
- U16 pad 3: /central_control_unit/water_sensors_logic/ws_rod_3 -> /central_control_unit/lightning/LEDS_CH34_5V
- U16 pad 4: /central_control_unit/water_sensors_logic/ws_rod_2 -> /central_control_unit/lightning/leds34_gnd
- U17 pad 5: /central_control_unit/230VAC/AC_DETECT -> /central_control_unit/ac_detect
- U3 pad 1: /central_control_unit/CAN/CAN_TX -> /central_control_unit/can_tx
- U3 pad 2: GND -> GND_LP
- U3 pad 4: /central_control_unit/CAN/CAN_RX -> /central_control_unit/can_rx
- U3 pad 5: Net-(U3-VIO) -> /central_control_unit/CAN/can_vio
- U3 pad 6: /central_control_unit/CAN/CAN_L -> /central_control_unit/can_term_r_dip_2
- U3 pad 8: /central_control_unit/CAN/CAN_SLEEP -> /central_control_unit/can_sleep
- U4 pad 1: GND_LP -> Net-(Q3-S)
- U4 pad 2: GND_LP -> Net-(Q4-D)
- U4 pad 3: +3.3V -> /central_control_unit/lightning/LEDS_CH12_5V
- U4 pad 4: /central_control_unit/strap pin -> /central_control_unit/lightning/leds12_gnd
- U6 pad 10: Net-(J5-Pin_1) -> /central_control_unit/digital_switching/CH1_OUT
- U6 pad 12: Net-(J5-Pin_1) -> /central_control_unit/digital_switching/CH1_OUT
- U6 pad 13: Net-(J5-Pin_1) -> /central_control_unit/digital_switching/CH1_OUT
- U6 pad 14: Net-(J5-Pin_1) -> /central_control_unit/digital_switching/CH1_OUT
- U6 pad 15: V_Bat -> +12V_HP
- U6 pad 8: Net-(J5-Pin_1) -> /central_control_unit/digital_switching/CH1_OUT
- U6 pad 9: Net-(J5-Pin_1) -> /central_control_unit/digital_switching/CH1_OUT
- U7 pad 10: Net-(J5-Pin_2) -> /central_control_unit/digital_switching/CH2_OUT
- U7 pad 12: Net-(J5-Pin_2) -> /central_control_unit/digital_switching/CH2_OUT
- U7 pad 13: Net-(J5-Pin_2) -> /central_control_unit/digital_switching/CH2_OUT
- U7 pad 14: Net-(J5-Pin_2) -> /central_control_unit/digital_switching/CH2_OUT
- U7 pad 15: V_Bat -> +12V_HP
- U7 pad 8: Net-(J5-Pin_2) -> /central_control_unit/digital_switching/CH2_OUT
- U7 pad 9: Net-(J5-Pin_2) -> /central_control_unit/digital_switching/CH2_OUT
- U8 pad 15: V_Bat -> +12V_HP
- U9 pad 10: Net-(J5-Pin_4) -> /central_control_unit/digital_switching/CH4_OUT
- U9 pad 12: Net-(J5-Pin_4) -> /central_control_unit/digital_switching/CH4_OUT
- U9 pad 13: Net-(J5-Pin_4) -> /central_control_unit/digital_switching/CH4_OUT
- U9 pad 14: Net-(J5-Pin_4) -> /central_control_unit/digital_switching/CH4_OUT
- U9 pad 15: V_Bat -> +12V_HP
- U9 pad 8: Net-(J5-Pin_4) -> /central_control_unit/digital_switching/CH4_OUT
- U9 pad 9: Net-(J5-Pin_4) -> /central_control_unit/digital_switching/CH4_OUT
Routing:
- net /central_control_unit/led_en: track 0.00 -> 109.7 mm
- net /central_control_unit/relay_out: track 0.00 -> 70.3 mm
- net /central_control_unit/ac_detect: track 0.00 -> 59.4 mm
- net /central_control_unit/water_sensors_logic/grey_water_probe: track 0.00 -> 37.2 mm, vias 0 -> 1
- net /central_control_unit/LED_CH4: track 0.00 -> 33.4 mm
- net /central_control_unit/water_sensors_logic/probe_4: track 0.00 -> 27.6 mm
- net /central_control_unit/LED_CH3: track 0.00 -> 25.5 mm
- net /central_control_unit/water_sensors_logic/probe_1: track 0.00 -> 19.2 mm
- net /central_control_unit/water_sensors_logic/ws_vref: track 0.00 -> 18.3 mm
- net /central_control_unit/water_sensors_logic/probe_3: track 0.00 -> 17.5 mm
- net /central_control_unit/WS_LVL_100: track 0.00 -> 17.3 mm
- net /central_control_unit/WS_LVL_75: track 0.00 -> 15.3 mm
- net /central_control_unit/LED_CH2: track 0.00 -> 14.6 mm
- net /central_control_unit/LED_CH1: track 0.00 -> 13.3 mm
- net /central_control_unit/water_sensors_logic/probe_2: track 0.00 -> 10.6 mm
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- added copper zone on B.Cu, net +12V_HP
- added copper zone on F.Cu, net +12V_HP
- added copper zone on B.Cu, net /central_control_unit/lightning/LEDS_CH12_5V
- added copper zone on F.Cu, net /central_control_unit/lightning/LEDS_CH12_5V
- added copper zone on B.Cu, net /central_control_unit/lightning/LEDS_CH34_5V
- added copper zone on F.Cu, net /central_control_unit/lightning/LEDS_CH34_5V
- added copper zone on B.Cu, net /central_control_unit/lightning/leds34_gnd
- added copper zone on F.Cu, net /central_control_unit/lightning/leds34_gnd
- added copper zone on B.Cu, net GND_HP
- removed copper zone on B.Cu, net V_Bat
- removed copper zone on F.Cu, net V_Bat
Other:
- board size 214.5 x 134.8 mm -> 201.6 x 244.9 mm
- board text removed: "RGB_LED logic"
- board text removed: "water_sensor_logic"
