File: electronics/230VAC.kicad_sch (KiCad schematic)
At the start: 11 parts, among them J21 Conn_01x02, J22 Conn_01x02, U13 CNY17-1, U17 H11AA1

Commit message: capacitors added. universal dc/dc converters
Parts:
- C9: footprint Capacitor_SMD:C_0805_2012Metric_Pad1.18x1.45mm_HandSolder -> Capacitor_SMD:C_0805_2012Metric
- R22, R25: footprint Resistor_SMD:R_0805_2012Metric_Pad1.20x1.40mm_HandSolder -> Resistor_SMD:R_0805_2012Metric
Changed lines of the file:
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@@
 	(label "N_230VAC"
 		(at 67.31 71.12 0)
-		(fields_autoplaced yes)
 		(effects
 			(font
@@
 	(label "P_230VAC"
 		(at 67.31 68.58 0)
-		(fields_autoplaced yes)
 		(effects
 			(font
@@
 	(label "V_Bat"
 		(at 110.49 96.52 0)
-		(fields_autoplaced yes)
 		(effects
 			(font
@@
 		(shape output)
 		(at 134.62 68.58 0)
-		(fields_autoplaced yes)
 		(effects
 			(font
@@
 		(shape input)
 		(at 57.15 107.95 180)
-		(fields_autoplaced yes)
 		(effects
 			(font
@@
 			)
 		)
-		(property "Footprint" "Resistor_SMD:R_0805_2012Metric_Pad1.20x1.40mm_HandSolder"
+		(property "Footprint" "Resistor_SMD:R_0805_2012Metric"
 			(at 119.38 66.548 90)
 			(effects
@@
 			)
 		)
-		(property "Footprint" "Capacitor_SMD:C_0805_2012Metric_Pad1.18x1.45mm_HandSolder"
+		(property "Footprint" "Capacitor_SMD:C_0805_2012Metric"
 			(at 123.19 71.12 0)
 			(effects
@@
 			)
 		)
-		(property "Footprint" "Resistor_SMD:R_0805_2012Metric_Pad1.20x1.40mm_HandSolder"
+		(property "Footprint" "Resistor_SMD:R_0805_2012Metric"
 			(at 68.58 109.728 90)
 			(effects
@@
 		(dnp no)
 		(fields_autoplaced yes)
-		(property "Reference" "#PWR045"
+		(property "Reference" "#PWR0101"
 			(at 115.57 63.5 0)
 			(effects
@@
 			(project "electronics"
 				(path "/eeb1234c-eae0-4ac6-a30d-2a978d66d889/04c402f1-b99a-4823-99a0-0c7312782f29/b07c78d9-bf9b-4530-b7c9-2098e4c7b5ee"
-					(reference "#PWR045")
-					(unit 1)
-				)
+					(reference "#PWR0101")
+					(unit 1)
+				)
