File: electronics/lightning.kicad_sch (KiCad schematic)
At the start: 19 parts, among them J1 leds_ch1, J20 leds_ch2, J26 leds_ch3, J27 leds_ch4, Q3 Q_PMOS_DGS, Q4 Q_NMOS_GDS, U2 ISO6740

Commit message: small progress on routing
Connections:
- net LEDS_CH12_5V: now also J1.3 (Pin_3), J20.3 (Pin_3); no longer J1.1 (Pin_1), J20.1 (Pin_1)
- net LEDS_CH34_5V: now also J26.3 (Pin_3), J27.3 (Pin_3); no longer J26.1 (Pin_1), J27.1 (Pin_1)
- net leds12_gnd: now also J1.1 (Pin_1), J20.1 (Pin_1); no longer J1.3 (Pin_3), J20.3 (Pin_3)
- net leds34_gnd: now also J26.1 (Pin_1), J27.1 (Pin_1); no longer J26.3 (Pin_3), J27.3 (Pin_3)
