File: electronics/lightning.kicad_sch (KiCad schematic)
At the start: 15 parts, among them J1 leds_ch1, J20 leds_ch2, J26 leds_ch3, J27 leds_ch4, Q6 Q_NMOS_GDS, U2 ISO6740

Commit message: progres on layouting
Parts:
- Q6: footprint Package_TO_SOT_SMD:TO-252-2 -> Package_TO_SOT_SMD:SOT-23
Changed lines of the file:
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@@
 	(label "LED_CH1"
 		(at 125.73 55.88 0)
-		(fields_autoplaced yes)
 		(effects
 			(font
@@
 	(label "LED_CH4"
 		(at 152.4 137.16 0)
-		(fields_autoplaced yes)
 		(effects
 			(font
@@
 	(label "LED_CH1"
 		(at 146.05 91.44 0)
-		(fields_autoplaced yes)
 		(effects
 			(font
@@
 	(label "LED_CH2"
 		(at 125.73 58.42 0)
-		(fields_autoplaced yes)
 		(effects
 			(font
@@
 	(label "LED_CH3"
 		(at 152.4 121.92 0)
-		(fields_autoplaced yes)
 		(effects
 			(font
@@
 	(label "LED_CH3"
 		(at 125.73 60.96 0)
-		(fields_autoplaced yes)
 		(effects
 			(font
@@
 	(label "LED_CH2"
 		(at 152.4 106.68 0)
-		(fields_autoplaced yes)
 		(effects
 			(font
@@
 	(label "LED_CH4"
 		(at 125.73 63.5 0)
-		(fields_autoplaced yes)
 		(effects
 			(font
@@
 		(shape input)
 		(at 81.28 60.96 180)
-		(fields_autoplaced yes)
 		(effects
 			(font
@@
 		(shape input)
 		(at 81.28 55.88 180)
-		(fields_autoplaced yes)
 		(effects
 			(font
@@
 		(shape input)
 		(at 81.28 63.5 180)
-		(fields_autoplaced yes)
 		(effects
 			(font
@@
 		(shape input)
 		(at 81.28 58.42 180)
-		(fields_autoplaced yes)
 		(effects
 			(font
@@
 		(shape input)
 		(at 27.94 139.7 180)
-		(fields_autoplaced yes)
 		(effects
 			(font
@@
 			)
 		)
-		(property "Footprint" "Package_TO_SOT_SMD:TO-252-2"
+		(property "Footprint" "Package_TO_SOT_SMD:SOT-23"
 			(at 64.77 134.62 0)
 			(effects

Commit message: layouting progress. some 3d models upload
Parts:
- removed C13: C_Polarized, Capacitor_THT:CP_Radial_D5.0mm_P2.50mm, symbol Device:C_Polarized
Changed lines of the file:
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@@
-	)
-	(junction
-		(at 120.65 111.76)
-		(diameter 0)
-		(color 0 0 0 0)
 	)
 	(junction
@@
 	)
 	(junction
-		(at 120.65 104.14)
-		(diameter 0)
-		(color 0 0 0 0)
-	)
-	(junction
 		(at 114.3 111.76)
 		(diameter 0)
@@
 	(wire
 		(pts
-			(xy 114.3 111.76) (xy 120.65 111.76)
-		)
-		(stroke
-			(width 0)
-			(type default)
-		)
-	)
-	(wire
-		(pts
 			(xy 53.34 149.86) (xy 53.34 156.21)
 		)
@@
 	(wire
 		(pts
-			(xy 120.65 111.76) (xy 133.35 111.76)
+			(xy 114.3 111.76) (xy 133.35 111.76)
 		)
 		(stroke
@@
 	(wire
 		(pts
-			(xy 114.3 104.14) (xy 120.65 104.14)
+			(xy 114.3 104.14) (xy 133.35 104.14)
 		)
 		(stroke
@@
 		(pts
 			(xy 146.05 109.22) (xy 161.29 109.22)
-		)
-		(stroke
-			(width 0)
-			(type default)
-		)
-	)
-	(wire
-		(pts
-			(xy 120.65 104.14) (xy 133.35 104.14)
 		)
 		(stroke
@@
 	(label "LED_CH1"
 		(at 125.73 55.88 0)
+		(fields_autoplaced yes)
 		(effects
 			(font
@@
 	(label "LED_CH4"
 		(at 152.4 137.16 0)
+		(fields_autoplaced yes)
 		(effects
 			(font
@@
 	(label "LED_CH1"
 		(at 146.05 91.44 0)
+		(fields_autoplaced yes)
 		(effects
 			(font
@@
 	(label "LED_CH2"
 		(at 125.73 58.42 0)
+		(fields_autoplaced yes)
 		(effects
 			(font
@@
 	(label "LED_CH3"
 		(at 152.4 121.92 0)
+		(fields_autoplaced yes)
 		(effects
 			(font
@@
 	(label "LED_CH3"
 		(at 125.73 60.96 0)
+		(fields_autoplaced yes)
 		(effects
 			(font
@@
 	(label "LED_CH2"
 		(at 152.4 106.68 0)
+		(fields_autoplaced yes)
 		(effects
 			(font
@@
 	(label "LED_CH4"
 		(at 125.73 63.5 0)
+		(fields_autoplaced yes)
 		(effects
 			(font
@@
 		(shape input)
 		(at 81.28 60.96 180)
+		(fields_autoplaced yes)
 		(effects
 			(font
@@
 		(shape input)
 		(at 81.28 55.88 180)
+		(fields_autoplaced yes)
 		(effects
 			(font
@@
 		(shape input)
 		(at 81.28 63.5 180)
+		(fields_autoplaced yes)
 		(effects
 			(font
@@
 		(shape input)
 		(at 81.28 58.42 180)
+		(fields_autoplaced yes)
 		(effects
 			(font
@@
 		(shape input)
 		(at 27.94 139.7 180)
+		(fields_autoplaced yes)
 		(effects
 			(font
@@
 					(unit 1)
 				)
-			)
-		)
-	)
-	(symbol
-		(lib_id "Device:C_Polarized")
-		(at 120.65 107.95 0)
-		(unit 1)
-		(exclude_from_sim no)
-		(in_bom yes)
-		(on_board yes)
-		(dnp yes)
-		(property "Reference" "C13"
-			(at 118.872 114.554 0)
-			(effects
-				(font
-					(size 1.27 1.27)
-				)
-				(justify left)
-			)
-		)
-		(property "Value" "C_Polarized"
-			(at 118.364 116.84 0)
-			(effects
-				(font
-					(size 1.27 1.27)
-				)
-				(justify left)
-			)
-		)
-		(property "Footprint" "Capacitor_THT:CP_Radial_D5.0mm_P2.50mm"
-			(at 121.6152 111.76 0)
-			(effects
-				(font
-					(size 1.27 1.27)
-				)
-				(hide yes)
-			)
-		)
-		(property "Datasheet" "~"
-			(at 120.65 107.95 0)
-			(effects
-				(font
-					(size 1.27 1.27)
-				)
-				(hide yes)
-			)
-		)
-		(property "Description" "Polarized capacitor"
-			(at 120.65 107.95 0)
-			(effects
-				(font
-					(size 1.27 1.27)
-				)
-				(hide yes)
-			)
-		)
-		(pin "2"
-		)
-		(pin "1"
-		)
-		(instances
-			(project "electronics"
-				(path "/eeb1234c-eae0-4ac6-a30d-2a978d66d889/04c402f1-b99a-4823-99a0-0c7312782f29/a6a65456-f9af-47c2-9797-83191f030e3b"
-					(reference "C13")
-					(unit 1)
-				)
